File: scoring/panel/pcb/target.sch (EAGLE design)
At the start: 16 parts, among them J1 AVRISP6_COMPACT, U1 ATTINY85-20SU

Commit message: Panel board: Update BOM with current macrofab part numbers in schematic and spreadsheet.
Parts:
- C1: DPN (none) -> 490-3897-1-ND; PRICE10 (none) -> 0.0440
- HIT: DPN (none) -> 160-1446-1-ND; PRICE10 (none) -> 0.238
- JP2: DPN 102-1170-ND -> 490-7800-ND; PRICE10 1.833 -> 0.794
- PWR: DPN (none) -> 160-1436-1-ND; PRICE10 (none) -> 0.218
- R1, R2: DPN P680ACT-ND -> P560GDKR-ND; PRICE10 0.0196 -> 0.00960
- R3, R4: DPN P10KACT-ND -> P10KGCT-ND; PRICE10 0.0196 -> 0.00960
- R6: DPN P100ACT-ND -> P100GCT-ND; PRICE10 0.0196 -> 0.00960
- R7: DPN (none) -> 2.0KGCT-ND; PRICE10 (none) -> 0.00960
- R8: DPN (none) -> P47GCT-ND; PRICE10 (none) -> 0.00960
- U$1: DPN (none) -> 455-1705-ND; PRICE10 (none) -> 0.173
Changed lines of the file:
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@@
 <part name="GND1" library="supply1" deviceset="GND" device=""/>
 <part name="R1" library="MF_Passives" deviceset="RESISTOR" device="_0603" value="560">
-<attribute name="DPN" value="P680ACT-ND"/>
-<attribute name="PRICE10" value="0.0196"/>
+<attribute name="DPN" value="P560GDKR-ND"/>
+<attribute name="PRICE10" value="0.00960"/>
 </part>
 <part name="R2" library="MF_Passives" deviceset="RESISTOR" device="_0603" value="560">
-<attribute name="DPN" value="P680ACT-ND"/>
-<attribute name="PRICE10" value="0.0196"/>
+<attribute name="DPN" value="P560GDKR-ND"/>
+<attribute name="PRICE10" value="0.00960"/>
 </part>
 <part name="R3" library="MF_Passives" deviceset="RESISTOR" device="_0603" value="10k">
-<attribute name="DPN" value="P10KACT-ND"/>
-<attribute name="PRICE10" value="0.0196"/>
+<attribute name="DPN" value="P10KGCT-ND"/>
+<attribute name="PRICE10" value="0.00960"/>
 </part>
 <part name="R4" library="MF_Passives" deviceset="RESISTOR" device="_0603" value="10k">
-<attribute name="DPN" value="P10KACT-ND"/>
-<attribute name="PRICE10" value="0.0196"/>
+<attribute name="DPN" value="P10KGCT-ND"/>
+<attribute name="PRICE10" value="0.00960"/>
 </part>
 <part name="GND2" library="supply1" deviceset="GND" device=""/>
@@
 <part name="P+5" library="supply1" deviceset="VCC" device=""/>
 <part name="JP2" library="pinhead" deviceset="PINHD-1X2" device="">
-<attribute name="DPN" value="102-1170-ND"/>
-<attribute name="PRICE10" value="1.833"/>
+<attribute name="DPN" value="490-7800-ND"/>
+<attribute name="PRICE10" value="0.794"/>
 </part>
 <part name="R5" library="MF_Passives" deviceset="RESISTOR" device="_0603" value="DNP"/>
 <part name="R6" library="MF_Passives" deviceset="RESISTOR" device="_0603" value="100">
-<attribute name="DPN" value="P100ACT-ND"/>
-<attribute name="PRICE10" value="0.0196"/>
+<attribute name="DPN" value="P100GCT-ND"/>
+<attribute name="PRICE10" value="0.00960"/>
 </part>
-<part name="PWR" library="MF_LEDs" deviceset="LED_SINGLE" device="_0603" value="RED"/>
-<part name="HIT" library="MF_LEDs" deviceset="LED_SINGLE" device="_0603" value="GRN"/>
-<part name="C1" library="MF_Passives" deviceset="CAPACITOR_NP" device="_0603" value="1uF"/>
-<part name="R7" library="MF_Passives" deviceset="RESISTOR" device="_0603" value="2k"/>
-<part name="U$1" library="jst-ph" deviceset="JST-PH3" device=""/>
-<part name="R8" library="MF_Passives" deviceset="RESISTOR" device="_0603" value="47"/>
+<part name="PWR" library="MF_LEDs" deviceset="LED_SINGLE" device="_0603" value="RED">
+<attribute name="DPN" value="160-1436-1-ND"/>
+<attribute name="PRICE10" value="0.218"/>
+</part>
+<part name="HIT" library="MF_LEDs" deviceset="LED_SINGLE" device="_0603" value="GRN">
+<attribute name="DPN" value="160-1446-1-ND"/>
+<attribute name="PRICE10" value="0.238"/>
+</part>
+<part name="C1" library="MF_Passives" deviceset="CAPACITOR_NP" device="_0603" value="1uF">
+<attribute name="DPN" value="490-3897-1-ND"/>
+<attribute name="PRICE10" value="0.0440"/>
+</part>
+<part name="R7" library="MF_Passives" deviceset="RESISTOR" device="_0603" value="2k">
+<attribute name="DPN" value="2.0KGCT-ND"/>
+<attribute name="PRICE10" value="0.00960"/>
+</part>
+<part name="U$1" library="jst-ph" deviceset="JST-PH3" device="">
+<attribute name="DPN" value="455-1705-ND"/>
+<attribute name="PRICE10" value="0.173"/>
+</part>
+<part name="R8" library="MF_Passives" deviceset="RESISTOR" device="_0603" value="47">
+<attribute name="DPN" value="P47GCT-ND"/>
+<attribute name="PRICE10" value="0.00960"/>
+</part>
 </parts>
 <sheets>
@@
 <attribute name="PRICE10" x="99.06" y="35.56" size="1.778" layer="96" rot="R90" display="off"/>
 </instance>
-<instance part="PWR" gate="G$1" x="-22.86" y="27.94" rot="R270"/>
-<instance part="HIT" gate="G$1" x="88.9" y="50.8" rot="R270"/>
-<instance part="C1" gate="G$1" x="-2.54" y="40.64"/>
-<instance part="R7" gate="G$1" x="78.74" y="50.8" rot="R90"/>
-<instance part="U$1" gate="A" x="109.22" y="73.66"/>
-<instance part="R8" gate="G$1" x="68.58" y="43.18"/>
+<instance part="PWR" gate="G$1" x="-22.86" y="27.94" rot="R270">
+<attribute name="DPN" x="-22.86" y="27.94" size="1.778" layer="96" rot="R270" display="off"/>
+<attribute name="PRICE10" x="-22.86" y="27.94" size="1.778" layer="96" rot="R270" display="off"/>
+</instance>
+<instance part="HIT" gate="G$1" x="88.9" y="50.8" rot="R270">
+<attribute name="DPN" x="88.9" y="50.8" size="1.778" layer="96" rot="R270" display="off"/>
+<attribute name="PRICE10" x="88.9" y="50.8" size="1.778" layer="96" rot="R270" display="off"/>
+</instance>
+<instance part="C1" gate="G$1" x="-2.54" y="40.64">
+<attribute name="DPN" x="-2.54" y="40.64" size="1.778" layer="96" display="off"/>
+<attribute name="PRICE10" x="-2.54" y="40.64" size="1.778" layer="96" display="off"/>
+</instance>
+<instance part="R7" gate="G$1" x="78.74" y="50.8" rot="R90">
+<attribute name="DPN" x="78.74" y="50.8" size="1.778" layer="96" rot="R90" display="off"/>
+<attribute name="PRICE10" x="78.74" y="50.8" size="1.778" layer="96" rot="R90" display="off"/>
+</instance>
+<instance part="U$1" gate="A" x="109.22" y="73.66">
+<attribute name="DPN" x="109.22" y="73.66" size="1.778" layer="96" display="off"/>
+<attribute name="PRICE10" x="109.22" y="73.66" size="1.778" layer="96" display="off"/>
+</instance>
+<instance part="R8" gate="G$1" x="68.58" y="43.18">
+<attribute name="DPN" x="68.58" y="43.18" size="1.778" layer="96" display="off"/>
+<attribute name="PRICE10" x="68.58" y="43.18" size="1.778" layer="96" display="off"/>
+</instance>
 </instances>
 <busses>
