File: hw/gimbal/pcb/gimbal.sch (EAGLE design)
At the start: 43 parts

Commit message: Progress on gimbal board.
Parts:
- added C14, C15: 0.01uF, rcl:C-USC0603
- added C16, C17, C20, C21, C22, C23, C24: 0.1uF, rcl:C-USC0603
- added C18, C19: 4.7uF, rcl:C-USC0603
- added C25, C26: 10pF, rcl:C-USC0603
- added R10, R8: 100k, rcl:R-US_R0603
- added R11, R9: 10k, rcl:R-US_R0603
- added R7: 10, rcl:R-US_R0603
- added U$16: (no value), gimbal:CRYSTALSMD5X3.2
- U$14: value (none) -> 2.2uH
Connections:
- new net BLDC_FAULT1: U$1.PC10/SPI3_SCK, U$5.FAULT/
- new net BLDC_FAULT2: U$1.PC9/TIM3_4/I2C3_SDA, U$6.FAULT/
- new net BLDC_RESET/: U$1.PC15, U$5.RESET/, U$6.RESET/
- new net BLDC_SLEEP/: U$1.PC14, U$5.SLEEP/, U$6.SLEEP/
- new net MOTOR1_EN: U$5.EN1, U$5.EN2, U$5.EN3
- new net MOTOR1_IN1: U$1.PC6/TIM3_1/UART6_TX, U$5.IN1
- new net MOTOR1_IN2: U$1.PC7/TIM3_2/SPI2_SCK/UART6_RX, U$5.IN2
- new net MOTOR1_IN3: U$1.PC8/TIM3_3, U$5.IN3
- new net MOTOR2_EN: U$6.EN1, U$6.EN2, U$6.EN3
- new net MOTOR2_IN1: U$1.PA0WKUP/TIM2_1/TIM5_1, U$6.IN1
- new net MOTOR2_IN2: U$1.PA1/TIM2_2/TIM5_2/SPI4_MOSI, U$6.IN2
- new net MOTOR2_IN3: U$1.PA2/TIM2_3/TIM5_3/TIM9_1/UART2_TX, U$6.IN3
- new net N$23: C18.1, U$1.VCAP1
- new net N$24: C24.1, U$1.NRST, U$9.5
- new net N$25: C14.1, U$6.CP1
- new net N$26: C14.2, U$6.CP2
- new net N$27: C15.2, U$5.CP2
- new net N$28: C15.1, U$5.CP1
- new net N$29: C16.2, U$5.VCP
- new net N$30: C17.2, U$6.VCP
- new net N$31: U$1.PA14/SWCLK, U$9.2
- new net N$32: U$1.PA13/SWDIO, U$9.4
- new net N$33: R7.2, U$1.BOOT0
- new net N$34: R8.1, R9.2, U$1.PC1
- new net N$35: C25.1, U$1.PH0, U$16.P$1
- new net N$36: C26.1, U$1.PH1, U$16.P$2
- new net N$38: R10.1, R11.2, U$1.PC2/SPI2_MISO
- new net SLAVE_RX: U$1.PB3/SWO/TIM2_2/SPI1_SCK/SPI3_SCK/UART1_RX/I2C2_SDA, U$8.3
- new net SLAVE_TX: U$1.PA15/TIM2_1/UART1_TX, U$8.2
- net +12V: now also C16.1, C17.1, R10.2, U$5.VM1, U$5.VM2, U$6.VM1, U$6.VM2
- net +3V3: now also C19.1, C20.1, C21.1, C22.1, C23.1, JP3.5, U$1.VBAT, U$1.VDD1, U$1.VDD2, U$1.VDD3, U$1.VDD4, U$1.VDDA, U$9.1
- net +8V: now also R8.2, U$8.4
- net AEG_PWM: now also U$1.PB0/TIM1_2N/TIM3_3/SPI5_SCK
- net AGITATOR_PWM: now also U$1.PB1/TIM1_3N/TIM3_4
- net AS5048_MISO: now also U$1.PA6/TIM3_1/SPI1_MISO; no longer U$1.PA6
- net AS5048_MOSI: now also U$1.PA7/TIM1_1N/TIM3_1/SPI1_MOSI; no longer U$1.PA7
- net AS5048_SCK: now also U$1.PA5/TIM2_1/SPI1_SCK; no longer U$1.PA5
- net BOOST_EN: now also U$1.PC11/SPI3_MISO
- net GND: now also C18.2, C19.2, C20.2, C21.2, C22.2, C23.2, C24.2, C25.2, C26.2, R11.1, R7.1, R9.1, U$1.VSS3, U$1.VSS4, U$16.P$3, U$5.GND1, U$5.GND2, U$5.GND3, U$5.PGND1, U$5.PGND2, U$5.PGND3, U$5.PPAD, U$6.GND1, U$6.GND2, U$6.GND3, U$6.PGND1, U$6.PGND2, U$6.PGND3, U$6.PPAD, U$8.1, U$9.3
- net LASER_EN: now also U$1.PB2
- net MOTOR_D1: now also U$1.PC12/SPI3_MOSI
- net MOTOR_FB: now also U$1.PC0
- net MOTOR_SF: now also U$1.PC13
- net PABS_SCL: now also U$1.PA8/TIM1_1/I2C3_SCL; no longer U$1.PB8
- net PABS_SDA: now also U$1.PB8/TIM4_3/TIM10_1/I2C1_SCL/SPI5_MOSI/I2C3_SDA; no longer U$1.PB9
- net PIMU_SCL: now also U$1.PB6/TIM4_1/I2C1_SCL/UART1_TX; no longer U$1.PA8
- net PIMU_SDA: now also U$1.PB7/TIM4_2/I2C1_SDA/UART1_RX; no longer U$1.PC9
- net SIMU_SCL: now also U$1.PB10/TIM2_3/I2C2_SCL/SPI2_SCK; no longer U$1.PB10
- net SIMU_SDA: now also U$1.PB9/TIM4_4/TIM11_1/I2C1_SDA/I2C2_SDA; no longer U$1.PB3
- net USB_DM: now also U$1.PA11/TIM1_4/SPI4_MISO/UART6_TX/USB_DM; no longer U$1.PA11
- net USB_DP: now also U$1.PA12/SPI5_MISO/UART6_RX/USB_DP; no longer U$1.PA12
- net USB_VBUS: now also U$1.PA9/TIM1_2/UART1_TX/USB_VBUS; no longer U$1.PA9
Other:
- moved on the sheet: U$10G$1, U$9

Commit message: gimbal board: Continued work: Updated all resistors and caps to the MF libraries.
Parts:
- removed C26: 10pF, rcl:C-USC0603
- added C27: 0.1uF, mfpassives:CAPACITOR_NP_0603
- added D1, D2, D3: (no value), mfleds:LED_SINGLE_0603
- added R12, R13, R14: 560, mfpassives:RESISTOR_0603
- added U$17: SLIDE_SWITCHJS_SUB_SWITCH, gimbal:SLIDE_SWITCHJS_SUB_SWITCH
- C11, C12, C13, C14, C15, C16, C17, C18, C19, C20, C21, C22, C23, C25, C4, C5: device rcl:C-USC0603 -> mfpassives:CAPACITOR_NP_0603
- C24: value 0.1uF -> 10pF; device rcl:C-USC0603 -> mfpassives:CAPACITOR_NP_0603
- R1, R10, R11, R2, R7, R8, R9: device rcl:R-US_R0603 -> mfpassives:RESISTOR_0603
- U$10: DPN (none) -> 609-4618-1-ND
- U$16: DPN (none) -> 535-9721-1-ND
Connections:
- new net N$37: D2.CATHODE, U$1.PB14/TIM1_2N/SPI2_MISO
- new net N$39: D1.ANODE, R12.P$1
- new net N$40: D2.ANODE, R13.P$1
- new net N$41: D3.ANODE, R14.P$1
- new net N$42: D3.CATHODE, U$1.PB13/TIM1_1N/SPI2_SCK/SPI4_SCK
- new net N$43: D1.CATHODE, U$1.PB15/TIM1_3N/SPI2_MOSI
- net +12V: now also C16.P$1, C27.P$1, R10.P$2; no longer C16.1, C17.1, R10.2
- net +3V3: now also C13.P$1, C17.P$1, C19.P$1, C20.P$1, C22.P$1, C23.P$1, R1.P$2, R12.P$2, R13.P$2, R14.P$2, U$17.1; no longer C13.1, C19.1, C20.1, C21.1, C22.1, C23.1, R1.2
- net +8V: now also R8.P$2; no longer R8.2
- net GND: now also C11.P$2, C12.P$2, C13.P$2, C17.P$2, C18.P$2, C19.P$2, C20.P$2, C21.P$2, C22.P$2, C23.P$2, C24.P$2, C25.P$2, C4.P$2, R11.P$1, R2.P$1, R7.P$1, R9.P$1, U$17.3; no longer C11.2, C12.2, C13.2, C18.2, C19.2, C20.2, C21.2, C22.2, C23.2, C24.2, C25.2, C26.2, C4.2, R11.1, R2.1, R7.1, R9.1
- net MOTOR_EN: now also U$1.PB12/SPI3_SCK, U$17.2
- net MOTOR_FB: now also R2.P$2; no longer R2.2
- net MOTOR_SF: now also R1.P$1; no longer R1.1
- net N$19: now also C11.P$1; no longer C11.1
- net N$21: now also C12.P$1; no longer C12.1
- net N$23: now also C18.P$1; no longer C18.1
- net N$24: now also C21.P$1; no longer C24.1
- net N$25: now also C14.P$1; no longer C14.1
- net N$26: now also C14.P$2; no longer C14.2
- net N$27: now also C15.P$2; no longer C15.2
- net N$28: now also C15.P$1; no longer C15.1
- net N$29: now also C27.P$2; no longer C16.2
- net N$30: now also C16.P$2; no longer C17.2
- net N$33: now also R7.P$2; no longer R7.2
- net N$34: now also R8.P$1, R9.P$2; no longer R8.1, R9.2
- net N$35: now also C24.P$1; no longer C25.1
- net N$36: now also C25.P$1; no longer C26.1
- net N$38: now also R10.P$1, R11.P$2; no longer R10.1, R11.2
- net N$4: now also C4.P$1, C5.P$1; no longer C4.1, C5.1
- net N$5: now also C5.P$2; no longer C5.2
Other:
- moved on the sheet: C11, C12, C13, C14, C15, C16, C17, C18, C19, C20, C21, C22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

Commit message: gimbal board: Finish updating the remaining larger caps to the macrofab library versions.
Parts:
- C1, C2, C3, C7: device rcl:C-USC1210 -> mfpassives:CAPACITOR_NP_1210
- C10, C6, C8: device rcl:C-USC1206 -> mfpassives:CAPACITOR_NP_1206
Connections:
- net +12V: now also C10.P$1; no longer C10.1
- net +3V3: now also C7.P$1; no longer C7.1
- net +8V: now also C6.P$1, C8.P$1; no longer C6.1, C8.1
- net GND: now also C1.P$2, C10.P$2, C2.P$2, C3.P$2, C6.P$2, C7.P$2, C8.P$2; no longer C1.2, C10.2, C2.2, C3.2, C6.2, C7.2, C8.2
- net N$4: now also C1.P$1, C2.P$1, C3.P$1; no longer C1.1, C2.1, C3.1
Other:
- moved on the sheet: C1, C10, C2, C3, C6, C7, C8, PABS, PIMU, SIMU, U$10G$1, U$11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

Commit message: gimbal board: Select a few parts, update TODO.
Parts:
- C18, C19: DPN (none) -> 311-1455-1-ND
Connections:
- removed net N$4: C1.P$1, C2.P$1, C3.P$1, C4.P$1, C5.P$1, U$2.VPWR
- net +8V: now also C1.P$1, C2.P$1, C3.P$1, C4.P$1, C5.P$1, U$2.VPWR
Changed lines of the file:
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@@
 <part name="C23" library="mfpassives" deviceset="CAPACITOR_NP" device="_0603" value="0.1uF"/>
 <part name="C20" library="mfpassives" deviceset="CAPACITOR_NP" device="_0603" value="0.1uF"/>
-<part name="C19" library="mfpassives" deviceset="CAPACITOR_NP" device="_0603" value="4.7uF"/>
-<part name="C18" library="mfpassives" deviceset="CAPACITOR_NP" device="_0603" value="4.7uF"/>
+<part name="C19" library="mfpassives" deviceset="CAPACITOR_NP" device="_0603" value="4.7uF">
+<attribute name="DPN" value="311-1455-1-ND"/>
+</part>
+<part name="C18" library="mfpassives" deviceset="CAPACITOR_NP" device="_0603" value="4.7uF">
+<attribute name="DPN" value="311-1455-1-ND"/>
+</part>
 <part name="C11" library="mfpassives" deviceset="CAPACITOR_NP" device="_0603" value="0.1uF"/>
 <part name="C12" library="mfpassives" deviceset="CAPACITOR_NP" device="_0603" value="0.047uF"/>
@@
 <attribute name="DPN" value="445-3955-1-ND"/>
 </part>
+<part name="SUPPLY5" library="supply2" deviceset="+8V" device=""/>
 </parts>
 <sheets>
@@
 <instance part="C23" gate="G$1" x="35.56" y="-243.84"/>
 <instance part="C20" gate="G$1" x="58.42" y="-243.84"/>
-<instance part="C19" gate="G$1" x="68.58" y="-243.84"/>
-<instance part="C18" gate="G$1" x="144.78" y="-248.92"/>
+<instance part="C19" gate="G$1" x="68.58" y="-243.84">
+<attribute name="DPN" x="68.58" y="-243.84" size="1.778" layer="96" display="off"/>
+</instance>
+<instance part="C18" gate="G$1" x="144.78" y="-248.92">
+<attribute name="DPN" x="144.78" y="-248.92" size="1.778" layer="96" display="off"/>
+</instance>
 <instance part="C11" gate="G$1" x="-15.24" y="-167.64"/>
 <instance part="C12" gate="G$1" x="-25.4" y="-167.64"/>
@@
 <attribute name="DPN" x="139.7" y="-152.4" size="1.778" layer="96" display="off"/>
 </instance>
+<instance part="SUPPLY5" gate="+8V" x="121.92" y="-121.92"/>
 </instances>
 <busses>
@@
 <pinref part="JP3" gate="A" pin="1"/>
 <wire x1="246.38" y1="-149.86" x2="259.08" y2="-149.86" width="0.1524" layer="91"/>
-</segment>
-</net>
-<net name="N$4" class="0">
-<segment>
-<pinref part="U$2" gate="G$1" pin="VPWR"/>
-<wire x1="228.6" y1="-139.7" x2="233.68" y2="-139.7" width="0.1524" layer="91"/>
-<wire x1="233.68" y1="-139.7" x2="233.68" y2="-124.46" width="0.1524" layer="91"/>
-<wire x1="233.68" y1="-124.46" x2="152.4" y2="-124.46" width="0.1524" layer="91"/>
-<wire x1="152.4" y1="-124.46" x2="139.7" y2="-124.46" width="0.1524" layer="91"/>
-<wire x1="139.7" y1="-124.46" x2="139.7" y2="-147.32" width="0.1524" layer="91"/>
-<wire x1="139.7" y1="-124.46" x2="129.54" y2="-124.46" width="0.1524" layer="91"/>
-<wire x1="129.54" y1="-124.46" x2="129.54" y2="-147.32" width="0.1524" layer="91"/>
-<junction x="139.7" y="-124.46"/>
-<wire x1="129.54" y1="-124.46" x2="116.84" y2="-124.46" width="0.1524" layer="91"/>
-<wire x1="116.84" y1="-124.46" x2="116.84" y2="-147.32" width="0.1524" layer="91"/>
-<junction x="129.54" y="-124.46"/>
-<wire x1="233.68" y1="-124.46" x2="241.3" y2="-124.46" width="0.1524" layer="91"/>
-<wire x1="241.3" y1="-124.46" x2="241.3" y2="-129.54" width="0.1524" layer="91"/>
-<junction x="233.68" y="-124.46"/>
-<pinref part="C5" gate="G$1" pin="P$1"/>
-<junction x="241.3" y="-129.54"/>
-<pinref part="C4" gate="G$1" pin="P$1"/>
-<wire x1="152.4" y1="-144.78" x2="152.4" y2="-124.46" width="0.1524" layer="91"/>
-<junction x="152.4" y="-124.46"/>
-<pinref part="C1" gate="G$1" pin="P$1"/>
-<pinref part="C2" gate="G$1" pin="P$1"/>
-<pinref part="C3" gate="G$1" pin="P$1"/>
 </segment>
 </net>
@@
 <wire x1="220.98" y1="-271.78" x2="220.98" y2="-274.32" width="0.1524" layer="91"/>
 </segment>
-</net>
+<segment>
+<pinref part="U$2" gate="G$1" pin="VPWR"/>
+<wire x1="228.6" y1="-139.7" x2="233.68" y2="-139.7" width="0.1524" layer="91"/>
+<wire x1="233.68" y1="-139.7" x2="233.68" y2="-124.46" width="0.1524" layer="91"/>
+<wire x1="233.68" y1="-124.46" x2="152.4" y2="-124.46" width="0.1524" layer="91"/>
+<wire x1="152.4" y1="-124.46" x2="139.7" y2="-124.46" width="0.1524" layer="91"/>
+<wire x1="139.7" y1="-124.46" x2="139.7" y2="-147.32" width="0.1524" layer="91"/>
+<wire x1="139.7" y1="-124.46" x2="129.54" y2="-124.46" width="0.1524" layer="91"/>
+<wire x1="129.54" y1="-124.46" x2="129.54" y2="-147.32" width="0.1524" layer="91"/>
+<junction x="139.7" y="-124.46"/>
+<wire x1="129.54" y1="-124.46" x2="121.92" y2="-124.46" width="0.1524" layer="91"/>
+<wire x1="121.92" y1="-124.46" x2="116.84" y2="-124.46" width="0.1524" layer="91"/>
+<wire x1="116.84" y1="-124.46" x2="116.84" y2="-147.32" width="0.1524" layer="91"/>
+<junction x="129.54" y="-124.46"/>
+<wire x1="233.68" y1="-124.46" x2="241.3" y2="-124.46" width="0.1524" layer="91"/>
+<wire x1="241.3" y1="-124.46" x2="241.3" y2="-129.54" width="0.1524" layer="91"/>
+<junction x="233.68" y="-124.46"/>
+<pinref part="C5" gate="G$1" pin="P$1"/>
+<junction x="241.3" y="-129.54"/>
+<pinref part="C4" gate="G$1" pin="P$1"/>
+<wire x1="152.4" y1="-144.78" x2="152.4" y2="-124.46" width="0.1524" layer="91"/>
+<junction x="152.4" y="-124.46"/>
+<pinref part="C1" gate="G$1" pin="P$1"/>
+<pinref part="C2" gate="G$1" pin="P$1"/>
+<pinref part="C3" gate="G$1" pin="P$1"/>
+<pinref part="SUPPLY5" gate="+8V" pin="+8V"/>
+<junction x="121.92" y="-124.46"/>
+</segment>
+</net>

Commit message: gimbal board: I2C pullups, AS50448A CS line, and more vias under the 12V boost regulator.
Parts:
- added R15, R16, R17, R18, R19, R20: 1.69k, mfpassives:RESISTOR_0603
Connections:
- new net AS5048_CS: U$1.PA4, U$3.CS/
- net +3V3: now also R15.P$2, R16.P$2, R17.P$2, R18.P$2, R19.P$2, R20.P$2
- net PABS_SCL: now also R20.P$1
- net PABS_SDA: now also R19.P$1
- net PIMU_SCL: now also R18.P$1
- net PIMU_SDA: now also R17.P$1
- net SIMU_SCL: now also R16.P$1
- net SIMU_SDA: now also R15.P$1
Other:
- moved on the sheet: PABS, SIMU

Commit message: gimbal board: Work towards naming all components.
Parts:
- J1: DPN (none) -> 455-2262-1-ND
- PABS, PIMU, SIMU: DPN (none) -> 455-1683-1-ND
- PGM: DPN (none) -> 455-1708-ND
- USBI: DPN (none) -> 455-1751-1-ND
- USBO: DPN (none) -> 455-1736-1-ND
- renumbered JP1 to M1, JP2 to M2, JP3 to J2, U$1 to U1, U$10 to USB, U$11 to MOUNT1, U$12 to MOUNT2, U$13 to L1, U$14 to L2, U$15 to D4, U$16 to Q1, U$17 to ARM, U$2 to U4, U$3 to U7, U$4 to U3, U$5 to U5, U$6 to U6, U$7 to U2, U$8 to J1, U$9 to PGM

Commit message: gimbal board: Rename all components and move around parts in the schematic to be slightly more organized.
Parts:
- removed C27: 0.1uF, mfpassives:CAPACITOR_NP_0603
- added C26: 0.1uF, mfpassives:CAPACITOR_NP_0603
- C1, C7: value 22uF 16V -> 4.7uF; device mfpassives:CAPACITOR_NP_1210 -> mfpassives:CAPACITOR_NP_0603; DPN 445-3955-1-ND -> 311-1455-1-ND
- C11, C17: value 0.1uF -> 22uF 16V; device mfpassives:CAPACITOR_NP_0603 -> mfpassives:CAPACITOR_NP_1210; DPN (none) -> 445-3955-1-ND
- C12: value 0.047uF -> 10uF; device mfpassives:CAPACITOR_NP_0603 -> mfpassives:CAPACITOR_NP_1206
- C13: value 0.1uF -> 0.047uF
- C14: value 0.01uF -> 0.1uF
- C15: value 0.01uF -> 100uF; device mfpassives:CAPACITOR_NP_0603 -> mfpassives:CAPACITOR_P_6.3MM
- C16: value 0.1uF -> 10uF; device mfpassives:CAPACITOR_NP_0603 -> mfpassives:CAPACITOR_NP_1206
- C18, C19: value 4.7uF -> 22uF 16V; device mfpassives:CAPACITOR_NP_0603 -> mfpassives:CAPACITOR_NP_1210; DPN 311-1455-1-ND -> 445-3955-1-ND
- C2, C3: value 22uF 16V -> 0.1uF; device mfpassives:CAPACITOR_NP_1210 -> mfpassives:CAPACITOR_NP_0603; DPN 445-3955-1-ND -> (none)
- C23: value 0.1uF -> 0.01uF
- C24: value 10pF -> 0.1uF
- C25: value 10pF -> 0.01uF
- C6: value 10uF -> 0.1uF; device mfpassives:CAPACITOR_NP_1206 -> mfpassives:CAPACITOR_NP_0603
- C8: value 10uF -> 10pF; device mfpassives:CAPACITOR_NP_1206 -> mfpassives:CAPACITOR_NP_0603
- C9: value 100uF -> 10pF; device mfpassives:CAPACITOR_P_6.3MM -> mfpassives:CAPACITOR_NP_0603
- R1: value 100k -> 10
- R10, R8: value 100k -> 10k
- R11: value 10k -> 78.4k
- R12: value 560 -> 1.87k
- R13: value 560 -> 100k
- R14: value 560 -> 220
- R2: value 220 -> 560
- R3: value 78.4k -> 560
- R4: value 1.87k -> 560
- R5: value 88k -> 100k
- R7: value 10 -> 100k
- R9: value 10k -> 88k
Connections:
- net +12V: now also C15.P$1, C22.P$1, C24.P$1, R7.P$2, R9.P$2; no longer C10.P$1, C27.P$1, C9.P$1, R10.P$2, R5.P$2
- net +3V3: now also C1.P$1, C11.P$1, C2.P$1, C26.P$1, C3.P$1, C4.P$1, C5.P$1, R2.P$2, R3.P$2, R4.P$2; no longer C13.P$1, C17.P$1, C19.P$1, C20.P$1, C22.P$1, C23.P$1, C7.P$1, R1.P$2, R12.P$2, R14.P$2
- net +8V: now also C10.P$1, C12.P$1, C17.P$1, C18.P$1, C19.P$1, C20.P$1, C21.P$1, R5.P$2; no longer C1.P$1, C2.P$1, C3.P$1, C4.P$1, C5.P$1, C6.P$1, C8.P$1, R8.P$2
- net GND: now also C14.P$2, C15.P$2, C16.P$2, C26.P$2, C5.P$2, R1.P$1, R10.P$1, R14.P$1, R8.P$1; no longer C21.P$2, C22.P$2, C23.P$2, C24.P$2, C25.P$2, R2.P$1, R3.P$1, R7.P$1, R9.P$1
- net MOTOR_FB: now also R14.P$2; no longer R2.P$2
- net MOTOR_SF: now also R13.P$1; no longer R1.P$1
- net N$18: now also R11.P$2; no longer R3.P$2
- net N$19: now also C14.P$1, R12.P$1; no longer C11.P$1, R4.P$1
- net N$20: now also R12.P$2; no longer R4.P$2
- net N$21: now also C13.P$1; no longer C12.P$1
- net N$22: now also R10.P$2, R9.P$1; no longer R5.P$1, R6.P$2
- net N$23: now also C7.P$1; no longer C18.P$1
- net N$24: now also C6.P$1; no longer C21.P$1
- net N$25: now also C25.P$1; no longer C14.P$1
- net N$26: now also C25.P$2; no longer C14.P$2
- net N$27: now also C23.P$2; no longer C15.P$2
- net N$28: now also C23.P$1; no longer C15.P$1
- net N$29: now also C22.P$2; no longer C27.P$2
- net N$30: now also C24.P$2; no longer C16.P$2
- net N$33: now also R1.P$2; no longer R7.P$2
- net N$34: now also R5.P$1, R6.P$2; no longer R8.P$1, R9.P$2
- net N$35: now also C8.P$1; no longer C24.P$1
- net N$36: now also C9.P$1; no longer C25.P$1
- net N$38: now also R7.P$1, R8.P$2; no longer R10.P$1, R11.P$2
- net N$39: now also R2.P$1; no longer R12.P$1
- net N$40: now also R3.P$1; no longer R13.P$1
- net N$41: now also R4.P$1; no longer R14.P$1
- net N$5: now also C21.P$2; no longer C5.P$2
- net PABS_SCL: now also R16.P$1; no longer R20.P$1
- net PABS_SDA: now also R15.P$1; no longer R19.P$1
- net SIMU_SCL: now also R20.P$1; no longer R16.P$1
- net SIMU_SDA: now also R19.P$1; no longer R15.P$1
Other:
- moved on the sheet: ARM, C1, C10, C11, C12, C13, C14, C16, C17, C18, C19, C2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
