File: hw/gimbal/pcb/gimbal.sch (EAGLE design)
At the start: 79 parts, among them J1 JST-XH4SMT_RA, U1 STM32F4R_64PIN, U2 TPS62172PWSON8, U3 TPS55330PQFN16, U4 MC33926, U5 DRV8313, U6 DRV8313, U7 AS5048A

Commit message: gimbal board: Final draft of all routing and silks.
Parts:
- added C27: 0.1uF, mfpassives:CAPACITOR_NP_0603
- renumbered PIMU to PI
Connections:
- net +3V3: now also C27.P$1
- net AS5048_CS: now also U1.PC11/SPI3_MISO; no longer U1.PA4
- net AS5048_MISO: now also U1.PB4/TIM3_1/SPI1_MISO/SPI3_MISO/I2C3_SDA; no longer U1.PA6/TIM3_1/SPI1_MISO
- net AS5048_MOSI: now also U1.PB5/TIM3_2/SPI1_MOSI/SPI3_MOSI; no longer U1.PA7/TIM1_1N/TIM3_1/SPI1_MOSI
- net AS5048_SCK: now also U1.PB3/SWO/TIM2_2/SPI1_SCK/SPI3_SCK/UART1_RX/I2C2_SDA; no longer U1.PA5/TIM2_1/SPI1_SCK
- net BLDC_FAULT1: now also U1.PA5/TIM2_1/SPI1_SCK; no longer U1.PC10/SPI3_SCK
- net BLDC_FAULT2: no longer U1.PC9/TIM3_4/I2C3_SDA
- net BLDC_RESET/: now also U1.PA7/TIM1_1N/TIM3_1/SPI1_MOSI; no longer U1.PC15
- net BLDC_SLEEP/: now also U1.PA6/TIM3_1/SPI1_MISO; no longer U1.PC14
- net BOOST_EN: now also U1.PC3/SPI2_MOSI; no longer U1.PC11/SPI3_MISO
- net GND: now also C27.P$2
- net MOTOR2_IN3: now also U1.PC9/TIM3_4/I2C3_SDA; no longer U1.PA2/TIM2_3/TIM5_3/TIM9_1/UART2_TX
- net SLAVE_RX: now also U1.PA3/TIM2_4/TIM5_4/TIM9_2/UART2_RX; no longer U1.PB3/SWO/TIM2_2/SPI1_SCK/SPI3_SCK/UART1_RX/I2C2_SDA
- net SLAVE_TX: now also U1.PA2/TIM2_3/TIM5_3/TIM9_1/UART2_TX; no longer U1.PA15/TIM2_1/UART1_TX
Changed lines of the file:
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@@
 <attribute name="DPN" value="455-1683-1-ND "/>
 </part>
-<part name="PIMU" library="gimbal" deviceset="JST-ZH4" device="">
+<part name="PI" library="gimbal" deviceset="JST-ZH4" device="">
 <attribute name="DPN" value="455-1683-1-ND"/>
 </part>
@@
 <part name="TP4" library="testpad" deviceset="TP" device="PAD1-13"/>
 <part name="U8" library="mfdiscrete" deviceset="N-CHANNEL_FET" device="_SOT-23-3"/>
+<part name="C27" library="mfpassives" deviceset="CAPACITOR_NP" device="_0603" value="0.1uF">
+<attribute name="AMFPN" value="MF-CAP-0603-0.1uF"/>
+</part>
 </parts>
 <sheets>
@@
 <attribute name="DPN" x="12.7" y="-325.12" size="1.778" layer="96" display="off"/>
 </instance>
-<instance part="PIMU" gate="G$1" x="73.66" y="-327.66">
+<instance part="PI" gate="G$1" x="73.66" y="-327.66">
 <attribute name="DPN" x="73.66" y="-327.66" size="1.778" layer="96" display="off"/>
 </instance>
@@
 <instance part="TP4" gate="G$1" x="81.28" y="40.64"/>
 <instance part="U8" gate="G$1" x="203.2" y="-63.5"/>
+<instance part="C27" gate="G$1" x="58.42" y="-325.12">
+<attribute name="AMFPN" x="58.42" y="-325.12" size="1.778" layer="96" display="off"/>
+</instance>
 </instances>
 <busses>
@@
 </segment>
 <segment>
-<pinref part="PIMU" gate="G$1" pin="4"/>
+<pinref part="PI" gate="G$1" pin="4"/>
 <pinref part="GND8" gate="1" pin="GND"/>
 <wire x1="81.28" y1="-330.2" x2="86.36" y2="-330.2" width="0.1524" layer="91"/>
@@
 <pinref part="GND9" gate="1" pin="GND"/>
 <wire x1="20.32" y1="-327.66" x2="25.4" y2="-327.66" width="0.1524" layer="91"/>
-<wire x1="25.4" y1="-327.66" x2="25.4" y2="-335.28" width="0.1524" layer="91"/>
+<wire x1="25.4" y1="-327.66" x2="25.4" y2="-330.2" width="0.1524" layer="91"/>
+<pinref part="C27" gate="G$1" pin="P$2"/>
+<wire x1="25.4" y1="-330.2" x2="25.4" y2="-335.28" width="0.1524" layer="91"/>
+<wire x1="58.42" y1="-330.2" x2="25.4" y2="-330.2" width="0.1524" layer="91"/>
+<junction x="25.4" y="-330.2"/>
 </segment>
 <segment>
@@
 <pinref part="R16" gate="G$1" pin="P$2"/>
 <wire x1="35.56" y1="-304.8" x2="35.56" y2="-307.34" width="0.1524" layer="91"/>
-</segment>
-<segment>
-<pinref part="PIMU" gate="G$1" pin="1"/>
+<pinref part="C27" gate="G$1" pin="P$1"/>
+<wire x1="25.4" y1="-320.04" x2="58.42" y2="-320.04" width="0.1524" layer="91"/>
+<junction x="25.4" y="-320.04"/>
+</segment>
+<segment>
+<pinref part="PI" gate="G$1" pin="1"/>
 <pinref part="+3V5" gate="G$1" pin="+3V3"/>
 <wire x1="81.28" y1="-322.58" x2="86.36" y2="-322.58" width="0.1524" layer="91"/>
@@
 </segment>
 <segment>
-<pinref part="U1" gate="G$1" pin="PC11/SPI3_MISO"/>
-<wire x1="170.18" y1="195.58" x2="213.36" y2="195.58" width="0.1524" layer="91"/>
-<label x="198.12" y="195.58" size="1.778" layer="95"/>
+<pinref part="U1" gate="G$1" pin="PC3/SPI2_MOSI"/>
+<wire x1="170.18" y1="215.9" x2="200.66" y2="215.9" width="0.1524" layer="91"/>
+<label x="193.04" y="215.9" size="1.778" layer="95"/>
 </segment>
 </net>
@@
 <net name="AS5048_SCK" class="0">
 <segment>
-<wire x1="48.26" y1="213.36" x2="5.08" y2="213.36" width="0.1524" layer="91"/>
-<label x="5.08" y="213.36" size="1.778" layer="95"/>
-<pinref part="U1" gate="G$1" pin="PA5/TIM2_1/SPI1_SCK"/>
-</segment>
-<segment>
 <pinref part="U7" gate="G$1" pin="CLK"/>
 <wire x1="116.84" y1="-246.38" x2="142.24" y2="-246.38" width="0.1524" layer="91"/>
 <label x="137.16" y="-246.38" size="1.778" layer="95"/>
 </segment>
+<segment>
+<pinref part="U1" gate="G$1" pin="PB3/SWO/TIM2_2/SPI1_SCK/SPI3_SCK/UART1_RX/I2C2_SDA"/>
+<wire x1="48.26" y1="175.26" x2="17.78" y2="175.26" width="0.1524" layer="91"/>
+<label x="17.78" y="175.26" size="1.778" layer="95"/>
+</segment>
 </net>
 <net name="AS5048_MISO" class="0">
@@
 </segment>
 <segment>
-<wire x1="48.26" y1="210.82" x2="5.08" y2="210.82" width="0.1524" layer="91"/>
-<label x="5.08" y="210.82" size="1.778" layer="95"/>
-<pinref part="U1" gate="G$1" pin="PA6/TIM3_1/SPI1_MISO"/>
+<pinref part="U1" gate="G$1" pin="PB4/TIM3_1/SPI1_MISO/SPI3_MISO/I2C3_SDA"/>
+<wire x1="48.26" y1="172.72" x2="17.78" y2="172.72" width="0.1524" layer="91"/>
+<label x="17.78" y="172.72" size="1.778" layer="95"/>
 </segment>
 </net>
 <net name="AS5048_MOSI" class="0">
-<segment>
-<wire x1="48.26" y1="208.28" x2="5.08" y2="208.28" width="0.1524" layer="91"/>
-<label x="5.08" y="208.28" size="1.778" layer="95"/>
-<pinref part="U1" gate="G$1" pin="PA7/TIM1_1N/TIM3_1/SPI1_MOSI"/>
-</segment>
 <segment>
 <pinref part="U7" gate="G$1" pin="MOSI"/>
@@
 <label x="137.16" y="-251.46" size="1.778" layer="95"/>
 </segment>
+<segment>
+<pinref part="U1" gate="G$1" pin="PB5/TIM3_2/SPI1_MOSI/SPI3_MOSI"/>
+<wire x1="48.26" y1="170.18" x2="17.78" y2="170.18" width="0.1524" layer="91"/>
+<label x="17.78" y="170.18" size="1.778" layer="95"/>
+</segment>
 </net>
 <net name="PIMU_SDA" class="0">
@@
 </segment>
 <segment>
-<pinref part="PIMU" gate="G$1" pin="2"/>
+<pinref part="PI" gate="G$1" pin="2"/>
 <wire x1="81.28" y1="-325.12" x2="91.44" y2="-325.12" width="0.1524" layer="91"/>
 <label x="99.06" y="-325.12" size="1.778" layer="95"/>
@@
 <net name="PIMU_SCL" class="0">
 <segment>
-<pinref part="PIMU" gate="G$1" pin="3"/>
+<pinref part="PI" gate="G$1" pin="3"/>
 <wire x1="81.28" y1="-327.66" x2="96.52" y2="-327.66" width="0.1524" layer="91"/>
 <label x="99.06" y="-327.66" size="1.778" layer="95"/>
@@
 </segment>
 <segment>
-<label x="17.78" y="187.96" size="1.778" layer="95"/>
-<wire x1="48.006" y1="187.96" x2="17.78" y2="187.96" width="0.1524" layer="91"/>
-<pinref part="U1" gate="G$1" pin="PA15/TIM2_1/UART1_TX"/>
+<pinref part="U1" gate="G$1" pin="PA2/TIM2_3/TIM5_3/TIM9_1/UART2_TX"/>
+<wire x1="48.26" y1="220.98" x2="12.7" y2="220.98" width="0.1524" layer="91"/>
+<label x="12.7" y="220.98" size="1.778" layer="95"/>
 </segment>
 </net>
@@
 </segment>
 <segment>
-<pinref part="U1" gate="G$1" pin="PB3/SWO/TIM2_2/SPI1_SCK/SPI3_SCK/UART1_RX/I2C2_SDA"/>
-<wire x1="48.26" y1="175.26" x2="17.78" y2="175.26" width="0.1524" layer="91"/>
-<label x="17.78" y="175.26" size="1.778" layer="95"/>
+<pinref part="U1" gate="G$1" pin="PA3/TIM2_4/TIM5_4/TIM9_2/UART2_RX"/>
+<wire x1="48.26" y1="218.44" x2="12.7" y2="218.44" width="0.1524" layer="91"/>
+<label x="12.7" y="218.44" size="1.778" layer="95"/>
 </segment>
 </net>
@@
 </segment>
 <segment>
-<pinref part="U1" gate="G$1" pin="PC15"/>
-<wire x1="170.18" y1="185.42" x2="210.82" y2="185.42" width="0.1524" layer="91"/>
-<label x="198.12" y="185.42" size="1.778" layer="95"/>
+<pinref part="U1" gate="G$1" pin="PA7/TIM1_1N/TIM3_1/SPI1_MOSI"/>
+<wire x1="48.26" y1="208.28" x2="7.62" y2="208.28" width="0.1524" layer="91"/>
+<label x="7.62" y="208.28" size="1.778" layer="95"/>
 </segment>
 </net>
@@
 </segment>
 <segment>
-<pinref part="U1" gate="G$1" pin="PC14"/>
-<wire x1="170.18" y1="187.96" x2="210.82" y2="187.96" width="0.1524" layer="91"/>
-<label x="198.12" y="187.96" size="1.778" layer="95"/>
+<pinref part="U1" gate="G$1" pin="PA6/TIM3_1/SPI1_MISO"/>
+<wire x1="48.26" y1="210.82" x2="7.62" y2="210.82" width="0.1524" layer="91"/>
+<label x="7.62" y="210.82" size="1.778" layer="95"/>
 </segment>
 </net>
@@
 </segment>
 <segment>
-<pinref part="U1" gate="G$1" pin="PC10/SPI3_SCK"/>
-<wire x1="170.18" y1="198.12" x2="213.36" y2="198.12" width="0.1524" layer="91"/>
-<label x="198.12" y="198.12" size="1.778" layer="95"/>
+<pinref part="U1" gate="G$1" pin="PA5/TIM2_1/SPI1_SCK"/>
+<wire x1="48.26" y1="213.36" x2="7.62" y2="213.36" width="0.1524" layer="91"/>
+<label x="7.62" y="213.36" size="1.778" layer="95"/>
 </segment>
 </net>
@@
 </segment>
 <segment>
-<pinref part="U1" gate="G$1" pin="PC9/TIM3_4/I2C3_SDA"/>
-<wire x1="170.18" y1="200.66" x2="213.36" y2="200.66" width="0.1524" layer="91"/>
-<label x="198.12" y="200.66" size="1.778" layer="95"/>
+<wire x1="48.26" y1="187.96" x2="17.78" y2="187.96" width="0.1524" layer="91"/>
+<label x="17.78" y="187.96" size="1.778" layer="95"/>
 </segment>
 </net>
@@
 </segment>
 <segment>
-<pinref part="U1" gate="G$1" pin="PA2/TIM2_3/TIM5_3/TIM9_1/UART2_TX"/>
-<wire x1="48.26" y1="220.98" x2="12.7" y2="220.98" width="0.1524" layer="91"/>
-<label x="12.7" y="220.98" size="1.778" layer="95"/>
+<pinref part="U1" gate="G$1" pin="PC9/TIM3_4/I2C3_SDA"/>
+<wire x1="170.18" y1="200.66" x2="200.66" y2="200.66" width="0.1524" layer="91"/>
+<label x="193.04" y="200.66" size="1.778" layer="95"/>
 </segment>
 </net>
@@
 <net name="AS5048_CS" class="0">
 <segment>
-<pinref part="U1" gate="G$1" pin="PA4"/>
-<wire x1="48.26" y1="215.9" x2="5.08" y2="215.9" width="0.1524" layer="91"/>
-<label x="5.08" y="215.9" size="1.778" layer="95"/>
-</segment>
-<segment>
 <pinref part="U7" gate="G$1" pin="CS/"/>
 <wire x1="116.84" y1="-243.84" x2="142.24" y2="-243.84" width="0.1524" layer="91"/>
 <label x="137.16" y="-243.84" size="1.778" layer="95"/>
 </segment>
-</net>
+<segment>
+<pinref part="U1" gate="G$1" pin="PC11/SPI3_MISO"/>
+<wire x1="170.18" y1="195.58" x2="213.36" y2="195.58" width="0.1524" layer="91"/>
+<label x="198.12" y="195.58" size="1.778" layer="95"/>
+</segment>
+</net>

Commit message: gimbal: Snapshot of board rework.  This doesn't currently autoroute, but has the motor enable lines connected to something.  It also has a lot of pin swaps in an attempt to clean up the routing.
Connections:
- removed net MOTOR1_EN: U5.EN1, U5.EN2, U5.EN3
- removed net MOTOR2_EN: U6.EN1, U6.EN2, U6.EN3
- new net BLDC_EN: U1.PD2, U5.EN1, U5.EN2, U5.EN3, U6.EN1, U6.EN2, U6.EN3
- net AS5048_CS: now also U1.PC15; no longer U1.PC11/SPI3_MISO
- net AS5048_MISO: now also U1.PC11/SPI3_MISO; no longer U1.PB4/TIM3_1/SPI1_MISO/SPI3_MISO/I2C3_SDA
- net AS5048_MOSI: now also U1.PC12/SPI3_MOSI; no longer U1.PB5/TIM3_2/SPI1_MOSI/SPI3_MOSI
- net AS5048_SCK: now also U1.PC10/SPI3_SCK; no longer U1.PB3/SWO/TIM2_2/SPI1_SCK/SPI3_SCK/UART1_RX/I2C2_SDA
- net LASER_EN: now also U1.PA10/TIM1_3/SPI5_MOSI/UART1_RX/USB_ID; no longer U1.PB2
- net MOTOR1_IN1: now also U1.PB3/SWO/TIM2_2/SPI1_SCK/SPI3_SCK/UART1_RX/I2C2_SDA; no longer U1.PC6/TIM3_1/UART6_TX
- net MOTOR1_IN2: now also U1.PB4/TIM3_1/SPI1_MISO/SPI3_MISO/I2C3_SDA; no longer U1.PC7/TIM3_2/SPI2_SCK/UART6_RX
- net MOTOR1_IN3: now also U1.PB5/TIM3_2/SPI1_MOSI/SPI3_MOSI; no longer U1.PC8/TIM3_3
- net MOTOR2_IN3: now also U1.PB8/TIM4_3/TIM10_1/I2C1_SCL/SPI5_MOSI/I2C3_SDA; no longer U1.PC9/TIM3_4/I2C3_SDA
- net MOTOR_D1: now also U1.PC14; no longer U1.PC12/SPI3_MOSI
- net PABS_SCL: now also U1.PB6/TIM4_1/I2C1_SCL/UART1_TX; no longer U1.PA8/TIM1_1/I2C3_SCL
- net PABS_SDA: now also U1.PB7/TIM4_2/I2C1_SDA/UART1_RX; no longer U1.PB8/TIM4_3/TIM10_1/I2C1_SCL/SPI5_MOSI/I2C3_SDA
- net PIMU_SCL: now also U1.PA8/TIM1_1/I2C3_SCL; no longer U1.PB6/TIM4_1/I2C1_SCL/UART1_TX
- net PIMU_SDA: now also U1.PC9/TIM3_4/I2C3_SDA; no longer U1.PB7/TIM4_2/I2C1_SDA/UART1_RX
Changed lines of the file:
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@@
 </segment>
 <segment>
-<pinref part="U1" gate="G$1" pin="PB2"/>
-<wire x1="17.78" y1="177.8" x2="48.26" y2="177.8" width="0.1524" layer="91"/>
-<label x="17.78" y="177.8" size="1.778" layer="95"/>
+<pinref part="U1" gate="G$1" pin="PA10/TIM1_3/SPI5_MOSI/UART1_RX/USB_ID"/>
+<wire x1="48.26" y1="200.66" x2="0" y2="200.66" width="0.1524" layer="91"/>
+<label x="0" y="200.66" size="1.778" layer="95"/>
 </segment>
 </net>
@@
 </segment>
 <segment>
-<pinref part="U1" gate="G$1" pin="PC12/SPI3_MOSI"/>
-<wire x1="170.18" y1="193.04" x2="213.36" y2="193.04" width="0.1524" layer="91"/>
-<label x="198.12" y="193.04" size="1.778" layer="95"/>
+<pinref part="U1" gate="G$1" pin="PC14"/>
+<wire x1="170.18" y1="187.96" x2="213.36" y2="187.96" width="0.1524" layer="91"/>
+<label x="198.12" y="187.96" size="1.778" layer="95"/>
 </segment>
 </net>
@@
 </segment>
 <segment>
-<pinref part="U1" gate="G$1" pin="PB3/SWO/TIM2_2/SPI1_SCK/SPI3_SCK/UART1_RX/I2C2_SDA"/>
-<wire x1="48.26" y1="175.26" x2="17.78" y2="175.26" width="0.1524" layer="91"/>
-<label x="17.78" y="175.26" size="1.778" layer="95"/>
+<pinref part="U1" gate="G$1" pin="PC10/SPI3_SCK"/>
+<wire x1="170.18" y1="198.12" x2="205.74" y2="198.12" width="0.1524" layer="91"/>
+<label x="195.58" y="198.12" size="1.778" layer="95"/>
 </segment>
 </net>
@@
 </segment>
 <segment>
-<pinref part="U1" gate="G$1" pin="PB4/TIM3_1/SPI1_MISO/SPI3_MISO/I2C3_SDA"/>
-<wire x1="48.26" y1="172.72" x2="17.78" y2="172.72" width="0.1524" layer="91"/>
-<label x="17.78" y="172.72" size="1.778" layer="95"/>
+<pinref part="U1" gate="G$1" pin="PC11/SPI3_MISO"/>
+<wire x1="170.18" y1="195.58" x2="205.74" y2="195.58" width="0.1524" layer="91"/>
+<label x="195.58" y="195.58" size="1.778" layer="95"/>
 </segment>
 </net>
@@
 </segment>
 <segment>
-<pinref part="U1" gate="G$1" pin="PB5/TIM3_2/SPI1_MOSI/SPI3_MOSI"/>
-<wire x1="48.26" y1="170.18" x2="17.78" y2="170.18" width="0.1524" layer="91"/>
-<label x="17.78" y="170.18" size="1.778" layer="95"/>
+<pinref part="U1" gate="G$1" pin="PC12/SPI3_MOSI"/>
+<wire x1="170.18" y1="193.04" x2="205.74" y2="193.04" width="0.1524" layer="91"/>
+<label x="195.58" y="193.04" size="1.778" layer="95"/>
 </segment>
 </net>
 <net name="PIMU_SDA" class="0">
-<segment>
-<wire x1="48.26" y1="165.1" x2="17.78" y2="165.1" width="0.1524" layer="91"/>
-<label x="17.78" y="165.1" size="1.778" layer="95"/>
-<pinref part="U1" gate="G$1" pin="PB7/TIM4_2/I2C1_SDA/UART1_RX"/>
-</segment>
 <segment>
 <pinref part="PI" gate="G$1" pin="2"/>
@@
 <junction x="91.44" y="-325.12"/>
 </segment>
+<segment>
+<pinref part="U1" gate="G$1" pin="PC9/TIM3_4/I2C3_SDA"/>
+<wire x1="170.18" y1="200.66" x2="200.66" y2="200.66" width="0.1524" layer="91"/>
+<label x="193.04" y="200.66" size="1.778" layer="95"/>
+</segment>
 </net>
 <net name="PIMU_SCL" class="0">
@@
 </segment>
 <segment>
-<pinref part="U1" gate="G$1" pin="PB6/TIM4_1/I2C1_SCL/UART1_TX"/>
-<wire x1="48.26" y1="167.64" x2="17.78" y2="167.64" width="0.1524" layer="91"/>
-<label x="17.78" y="167.64" size="1.778" layer="95"/>
+<pinref part="U1" gate="G$1" pin="PA8/TIM1_1/I2C3_SCL"/>
+<wire x1="48.26" y1="205.74" x2="5.08" y2="205.74" width="0.1524" layer="91"/>
+<label x="5.08" y="205.74" size="1.778" layer="95"/>
 </segment>
 </net>
@@
 </segment>
 <segment>
-<pinref part="U1" gate="G$1" pin="PA8/TIM1_1/I2C3_SCL"/>
-<wire x1="48.26" y1="205.74" x2="5.08" y2="205.74" width="0.1524" layer="91"/>
-<label x="5.08" y="205.74" size="1.778" layer="95"/>
+<pinref part="U1" gate="G$1" pin="PB6/TIM4_1/I2C1_SCL/UART1_TX"/>
+<wire x1="48.26" y1="167.64" x2="17.78" y2="167.64" width="0.1524" layer="91"/>
+<label x="17.78" y="167.64" size="1.778" layer="95"/>
 </segment>
 </net>
@@
 </segment>
 <segment>
-<pinref part="U1" gate="G$1" pin="PB8/TIM4_3/TIM10_1/I2C1_SCL/SPI5_MOSI/I2C3_SDA"/>
-<wire x1="48.26" y1="162.56" x2="17.78" y2="162.56" width="0.1524" layer="91"/>
-<label x="17.78" y="162.56" size="1.778" layer="95"/>
+<wire x1="48.26" y1="165.1" x2="17.78" y2="165.1" width="0.1524" layer="91"/>
+<label x="17.78" y="165.1" size="1.778" layer="95"/>
+<pinref part="U1" gate="G$1" pin="PB7/TIM4_2/I2C1_SDA/UART1_RX"/>
 </segment>
 </net>
@@
 </segment>
 </net>
-<net name="MOTOR1_EN" class="0">
-<segment>
-<pinref part="U5" gate="G$1" pin="EN1"/>
-<wire x1="17.78" y1="-175.26" x2="-20.32" y2="-175.26" width="0.1524" layer="91"/>
-<label x="-20.32" y="-175.26" size="1.778" layer="95"/>
-</segment>
-<segment>
-<pinref part="U5" gate="G$1" pin="EN2"/>
-<wire x1="17.78" y1="-182.88" x2="-22.86" y2="-182.88" width="0.1524" layer="91"/>
-<label x="-20.32" y="-182.88" size="1.778" layer="95"/>
-</segment>
-<segment>
-<pinref part="U5" gate="G$1" pin="EN3"/>
-<wire x1="17.78" y1="-190.5" x2="-20.32" y2="-190.5" width="0.1524" layer="91"/>
-<label x="-20.32" y="-190.5" size="1.778" layer="95"/>
-</segment>
-</net>
-<net name="MOTOR2_EN" class="0">
-<segment>
-<pinref part="U6" gate="G$1" pin="EN1"/>
-<wire x1="177.8" y1="-177.8" x2="139.7" y2="-177.8" width="0.1524" layer="91"/>
-<label x="139.7" y="-177.8" size="1.778" layer="95"/>
-</segment>
-<segment>
-<pinref part="U6" gate="G$1" pin="EN2"/>
-<wire x1="177.8" y1="-185.42" x2="139.7" y2="-185.42" width="0.1524" layer="91"/>
-<label x="139.7" y="-185.42" size="1.778" layer="95"/>
-</segment>
-<segment>
-<pinref part="U6" gate="G$1" pin="EN3"/>
-<wire x1="177.8" y1="-193.04" x2="139.7" y2="-193.04" width="0.1524" layer="91"/>
-<label x="139.7" y="-193.04" size="1.778" layer="95"/>
-</segment>
-</net>
 <net name="MOTOR1_IN1" class="0">
 <segment>
@@
 </segment>
 <segment>
-<pinref part="U1" gate="G$1" pin="PC6/TIM3_1/UART6_TX"/>
-<wire x1="170.18" y1="208.28" x2="200.66" y2="208.28" width="0.1524" layer="91"/>
-<label x="193.04" y="208.28" size="1.778" layer="95"/>
+<pinref part="U1" gate="G$1" pin="PB3/SWO/TIM2_2/SPI1_SCK/SPI3_SCK/UART1_RX/I2C2_SDA"/>
+<wire x1="48.26" y1="175.26" x2="12.7" y2="175.26" width="0.1524" layer="91"/>
+<label x="12.7" y="175.26" size="1.778" layer="95"/>
 </segment>
 </net>
@@
 </segment>
 <segment>
-<pinref part="U1" gate="G$1" pin="PC7/TIM3_2/SPI2_SCK/UART6_RX"/>
-<wire x1="170.18" y1="205.74" x2="200.66" y2="205.74" width="0.1524" layer="91"/>
-<label x="193.04" y="205.74" size="1.778" layer="95"/>
+<pinref part="U1" gate="G$1" pin="PB4/TIM3_1/SPI1_MISO/SPI3_MISO/I2C3_SDA"/>
+<wire x1="48.26" y1="172.72" x2="12.7" y2="172.72" width="0.1524" layer="91"/>
+<label x="12.7" y="172.72" size="1.778" layer="95"/>
 </segment>
 </net>
@@
 </segment>
 <segment>
-<pinref part="U1" gate="G$1" pin="PC8/TIM3_3"/>
-<wire x1="170.18" y1="203.2" x2="200.66" y2="203.2" width="0.1524" layer="91"/>
-<label x="193.04" y="203.2" size="1.778" layer="95"/>
+<pinref part="U1" gate="G$1" pin="PB5/TIM3_2/SPI1_MOSI/SPI3_MOSI"/>
+<wire x1="48.26" y1="170.18" x2="12.7" y2="170.18" width="0.1524" layer="91"/>
+<label x="12.7" y="170.18" size="1.778" layer="95"/>
 </segment>
 </net>
@@
 </segment>
 <segment>
-<pinref part="U1" gate="G$1" pin="PC9/TIM3_4/I2C3_SDA"/>
-<wire x1="170.18" y1="200.66" x2="200.66" y2="200.66" width="0.1524" layer="91"/>
-<label x="193.04" y="200.66" size="1.778" layer="95"/>
+<pinref part="U1" gate="G$1" pin="PB8/TIM4_3/TIM10_1/I2C1_SCL/SPI5_MOSI/I2C3_SDA"/>
+<wire x1="48.26" y1="162.56" x2="12.7" y2="162.56" width="0.1524" layer="91"/>
+<label x="12.7" y="162.56" size="1.778" layer="95"/>
 </segment>
 </net>
@@
 </segment>
 <segment>
-<pinref part="U1" gate="G$1" pin="PC11/SPI3_MISO"/>
-<wire x1="170.18" y1="195.58" x2="213.36" y2="195.58" width="0.1524" layer="91"/>
-<label x="198.12" y="195.58" size="1.778" layer="95"/>
-</segment>
-</net>
+<pinref part="U1" gate="G$1" pin="PC15"/>
+<wire x1="170.18" y1="185.42" x2="213.36" y2="185.42" width="0.1524" layer="91"/>
+<label x="198.12" y="185.42" size="1.778" layer="95"/>
+</segment>
+</net>
+<net name="BLDC_EN" class="0">
+<segment>
+<pinref part="U5" gate="G$1" pin="EN1"/>
+<wire x1="17.78" y1="-175.26" x2="-20.32" y2="-175.26" width="0.1524" layer="91"/>
+<label x="-20.32" y="-175.26" size="1.778" layer="95"/>
+</segment>
+<segment>
+<pinref part="U5" gate="G$1" pin="EN3"/>
+<wire x1="17.78" y1="-190.5" x2="-20.32" y2="-190.5" width="0.1524" layer="91"/>
+<label x="-20.32" y="-190.5" size="1.778" layer="95"/>
+</segment>
+<segment>
+<pinref part="U5" gate="G$1" pin="EN2"/>
+<wire x1="17.78" y1="-182.88" x2="-22.86" y2="-182.88" width="0.1524" layer="91"/>
+<label x="-20.32" y="-182.88" size="1.778" layer="95"/>
+</segment>
+<segment>
+<pinref part="U6" gate="G$1" pin="EN1"/>
+<wire x1="177.8" y1="-177.8" x2="139.7" y2="-177.8" width="0.1524" layer="91"/>
+<label x="139.7" y="-177.8" size="1.778" layer="95"/>
+</segment>
+<segment>
+<pinref part="U6" gate="G$1" pin="EN2"/>
+<wire x1="177.8" y1="-185.42" x2="139.7" y2="-185.42" width="0.1524" layer="91"/>
+<label x="139.7" y="-185.42" size="1.778" layer="95"/>
+</segment>
+<segment>
+<pinref part="U6" gate="G$1" pin="EN3"/>
+<wire x1="177.8" y1="-193.04" x2="139.7" y2="-193.04" width="0.1524" layer="91"/>
+<label x="139.7" y="-193.04" size="1.778" layer="95"/>
+</segment>
+<segment>
+<pinref part="U1" gate="G$1" pin="PD2"/>
+<wire x1="170.18" y1="180.34" x2="213.36" y2="180.34" width="0.1524" layer="91"/>
+<label x="198.12" y="180.34" size="1.778" layer="95"/>
+</segment>
+</net>
