File: hw/joule_shield_v1/pcb/joule_shield.sch (EAGLE design)
At the start: 128 parts, among them J1 MF-CON-MICROUSB-RIGHT, J4 USB_AUSB_A_SMT_RA, J5 JST-ZH5SMT_RA, J6 INTEL_JOULE_J6, J7 INTEL_JOULE_J7, J8 DM3ATDM3AT, Q1 NFETEMT3F, Q2 NFETEMT3F, Q3 NFETEMT3F, Q4 NFETEMT3F, Q5 NFETEMT3F, SW1 MF-SW-TACT-4.2MM, SW2 MF-SW-TACT-4.2MM, SW3 MF-SW-TACT-4.2MM, U1 BQ25892PWQFN-24, U10 FT231XQFN-20, U2 FAN8623WLCSP16, U5 TPS2553PWSON-6, U6 TPS2553PWSON-6, U7 SINGLE-BIT_BUS_TRANSCEIVER, U8 SINGLE-BIT_BUS_TRANSCEIVER, U9 SN74AVCA406L

Commit message: joule shield snapshot
Parts:
- removed C19: 22uF, mf_passives:CAPACITOR_NP_0603
- renumbered SW1 to PWR, SW2 to DNX, SW3 to BTN
Connections:
- net GND: now also U$48.P$1, U$49.P$1, U$50.P$1, U$51.P$1; no longer C19.P$2
- net V3P3V: no longer C19.P$1
Changed lines of the file:
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@@
-<attribute name="MPN" value="CL10A226MP8NUNE"/>
-</part>
-<part name="C19" library="mf_passives" deviceset="CAPACITOR_NP" device="_0603" value="22uF">
-<attribute name="DPN" value="1276-1274-1-ND"/>
 <attribute name="MPN" value="CL10A226MP8NUNE"/>
 </part>
@@
 <attribute name="MPN" value="MF-RES-0603-27"/>
 </part>
-<part name="SW1" library="mf_switches" deviceset="TACT" device="_4.2MM" value="MF-SW-TACT-4.2MM"/>
-<part name="SW2" library="mf_switches" deviceset="TACT" device="_4.2MM" value="MF-SW-TACT-4.2MM"/>
-<part name="SW3" library="mf_switches" deviceset="TACT" device="_4.2MM" value="MF-SW-TACT-4.2MM"/>
+<part name="PWR" library="mf_switches" deviceset="TACT" device="_4.2MM" value="MF-SW-TACT-4.2MM"/>
+<part name="DNX" library="mf_switches" deviceset="TACT" device="_4.2MM" value="MF-SW-TACT-4.2MM"/>
+<part name="BTN" library="mf_switches" deviceset="TACT" device="_4.2MM" value="MF-SW-TACT-4.2MM"/>
 <part name="GND48" library="supply1" deviceset="GND" device=""/>
 <part name="D5" library="joule_shield" deviceset="ESD_DIODE" device="M1005">
@@
 <attribute name="POPULATE" value="1"/>
 </part>
+<part name="GND12" library="supply1" deviceset="GND" device=""/>
 </parts>
 <sheets>
@@
 </instance>
 <instance part="U$58" gate="G$1" x="-10.16" y="172.72"/>
+<instance part="GND12" gate="1" x="-25.4" y="-35.56"/>
 </instances>
 <busses>
@@
 <pinref part="J5" gate="G$1" pin="5"/>
 <wire x1="287.02" y1="78.74" x2="294.64" y2="78.74" width="0.1524" layer="91"/>
+</segment>
+<segment>
+<pinref part="GND12" gate="1" pin="GND"/>
+<pinref part="U$48" gate="G$1" pin="P$1"/>
+<wire x1="-25.4" y1="-33.02" x2="-25.4" y2="-30.48" width="0.1524" layer="91"/>
+<pinref part="U$49" gate="G$1" pin="P$1"/>
+<wire x1="-25.4" y1="-30.48" x2="-25.4" y2="-27.94" width="0.1524" layer="91"/>
+<wire x1="-25.4" y1="-30.48" x2="-7.62" y2="-30.48" width="0.1524" layer="91"/>
+<wire x1="-7.62" y1="-30.48" x2="-7.62" y2="-27.94" width="0.1524" layer="91"/>
+<junction x="-25.4" y="-30.48"/>
+<pinref part="U$50" gate="G$1" pin="P$1"/>
+<wire x1="-7.62" y1="-30.48" x2="10.16" y2="-30.48" width="0.1524" layer="91"/>
+<wire x1="10.16" y1="-30.48" x2="10.16" y2="-27.94" width="0.1524" layer="91"/>
+<junction x="-7.62" y="-30.48"/>
+<pinref part="U$51" gate="G$1" pin="P$1"/>
+<wire x1="10.16" y1="-30.48" x2="27.94" y2="-30.48" width="0.1524" layer="91"/>
+<wire x1="27.94" y1="-30.48" x2="27.94" y2="-27.94" width="0.1524" layer="91"/>
+<junction x="10.16" y="-30.48"/>
 </segment>
 </net>
@@
 <attribute name="DPN" x="68.58" y="119.38" size="1.778" layer="96" display="off"/>
 </instance>
-<instance part="C19" gate="G$1" x="76.2" y="119.38">
-<attribute name="DPN" x="76.2" y="119.38" size="1.778" layer="96" display="off"/>
-</instance>
 <instance part="C20" gate="G$1" x="86.36" y="119.38"/>
 <instance part="GND15" gate="1" x="71.12" y="111.76"/>
@@
 <wire x1="68.58" y1="116.84" x2="68.58" y2="114.3" width="0.1524" layer="91"/>
 <junction x="68.58" y="114.3"/>
-<pinref part="C19" gate="G$1" pin="P$2"/>
-<wire x1="71.12" y1="114.3" x2="76.2" y2="114.3" width="0.1524" layer="91"/>
-<wire x1="76.2" y1="114.3" x2="76.2" y2="116.84" width="0.1524" layer="91"/>
 <junction x="71.12" y="114.3"/>
 <pinref part="C20" gate="G$1" pin="P$2"/>
-<wire x1="76.2" y1="114.3" x2="86.36" y2="114.3" width="0.1524" layer="91"/>
+<wire x1="71.12" y1="114.3" x2="86.36" y2="114.3" width="0.1524" layer="91"/>
 <wire x1="86.36" y1="114.3" x2="86.36" y2="116.84" width="0.1524" layer="91"/>
-<junction x="76.2" y="114.3"/>
 </segment>
 </net>
@@
 <wire x1="68.58" y1="124.46" x2="68.58" y2="121.92" width="0.1524" layer="91"/>
 <junction x="68.58" y="124.46"/>
-<pinref part="C19" gate="G$1" pin="P$1"/>
-<wire x1="76.2" y1="124.46" x2="76.2" y2="121.92" width="0.1524" layer="91"/>
 <junction x="76.2" y="124.46"/>
 <pinref part="C20" gate="G$1" pin="P$1"/>
@@
 <instance part="R27" gate="G$1" x="180.34" y="55.88"/>
 <instance part="GND44" gate="1" x="149.86" y="20.32"/>
-<instance part="SW1" gate="G$1" x="17.78" y="124.46"/>
-<instance part="SW2" gate="G$1" x="88.9" y="124.46"/>
-<instance part="SW3" gate="G$1" x="162.56" y="124.46"/>
+<instance part="PWR" gate="G$1" x="17.78" y="124.46"/>
+<instance part="DNX" gate="G$1" x="88.9" y="124.46"/>
+<instance part="BTN" gate="G$1" x="162.56" y="124.46"/>
 <instance part="GND48" gate="1" x="10.16" y="99.06"/>
 <instance part="D5" gate="G$1" x="33.02" y="116.84" rot="R90">
@@
 <pinref part="GND48" gate="1" pin="GND"/>
 <wire x1="10.16" y1="101.6" x2="10.16" y2="104.14" width="0.1524" layer="91"/>
-<pinref part="SW1" gate="G$1" pin="P$3"/>
+<pinref part="PWR" gate="G$1" pin="P$3"/>
 <wire x1="10.16" y1="104.14" x2="10.16" y2="121.92" width="0.1524" layer="91"/>
 <wire x1="10.16" y1="121.92" x2="15.24" y2="121.92" width="0.1524" layer="91"/>
@@
 </segment>
 <segment>
-<pinref part="SW3" gate="G$1" pin="P$3"/>
+<pinref part="BTN" gate="G$1" pin="P$3"/>
 <wire x1="160.02" y1="121.92" x2="154.94" y2="121.92" width="0.1524" layer="91"/>
 <pinref part="GND50" gate="1" pin="GND"/>
@@
 <net name="PMIC_PWRBTN_N" class="0">
 <segment>
-<pinref part="SW1" gate="G$1" pin="P$2"/>
+<pinref part="PWR" gate="G$1" pin="P$2"/>
 <pinref part="D5" gate="G$1" pin="P$2"/>
 <wire x1="20.32" y1="127" x2="33.02" y2="127" width="0.1524" layer="91"/>
@@
 <pinref part="R31" gate="G$1" pin="P$2"/>
 <wire x1="73.66" y1="124.46" x2="73.66" y2="121.92" width="0.1524" layer="91"/>
-<pinref part="SW2" gate="G$1" pin="P$3"/>
+<pinref part="DNX" gate="G$1" pin="P$3"/>
 <wire x1="73.66" y1="121.92" x2="86.36" y2="121.92" width="0.1524" layer="91"/>
 </segment>
@@
 <net name="UART2_TX" class="0">
 <segment>
-<pinref part="SW2" gate="G$1" pin="P$2"/>
+<pinref part="DNX" gate="G$1" pin="P$2"/>
 <pinref part="D6" gate="G$1" pin="P$2"/>
 <wire x1="91.44" y1="127" x2="106.68" y2="127" width="0.1524" layer="91"/>
@@
 <pinref part="R32" gate="G$1" pin="P$2"/>
 <wire x1="144.78" y1="129.54" x2="144.78" y2="127" width="0.1524" layer="91"/>
-<pinref part="SW3" gate="G$1" pin="P$1"/>
+<pinref part="BTN" gate="G$1" pin="P$1"/>
 <wire x1="144.78" y1="127" x2="160.02" y2="127" width="0.1524" layer="91"/>
 </segment>
@@
 <net name="BTN_N" class="0">
 <segment>
-<pinref part="SW3" gate="G$1" pin="P$2"/>
+<pinref part="BTN" gate="G$1" pin="P$2"/>
 <pinref part="D7" gate="G$1" pin="P$2"/>
 <wire x1="165.1" y1="127" x2="177.8" y2="127" width="0.1524" layer="91"/>

Commit message: joule shield checkpoint
Parts:
- added LED1, SYS: MF-LED-0603-RED, mf_leds:LED_SINGLE-0603-RED
- added R13: 0, mf_passives:RESISTOR_0603
- D1, D8: value MF-LED-0603-RED -> MF-DIO-SOD123-BAT42; device mf_leds:LED_SINGLE-0603-RED -> mf_discrete_semiconductor:DIODES_BAT42_SOD-123
- renumbered D10 to LED3, D9 to LED2
Connections:
- new net N$10: J6.USB2_ID_PMIC, R13.P$1
- new net N$16: D1.ANODE, FB3.P$2
- net GND: now also R13.P$2
- net N$1: now also SYS.ANODE; no longer D1.ANODE
- net N$49: now also D1.CATHODE, D8.CATHODE; no longer FB3.P$2
- net N$58: now also LED1.ANODE; no longer D8.ANODE
- net N$59: now also LED1.CATHODE; no longer D8.CATHODE
- net N$6: now also SYS.CATHODE; no longer D1.CATHODE
- net V5P0V: now also D8.ANODE
Other:
- moved on the sheet: FB3
Changed lines of the file:
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@@
 <attribute name="MPN" value="MF-RES-0603-100K"/>
 </part>
-<part name="D1" library="mf_leds" deviceset="LED_SINGLE" device="-0603-RED" value="MF-LED-0603-RED"/>
+<part name="SYS" library="mf_leds" deviceset="LED_SINGLE" device="-0603-RED" value="MF-LED-0603-RED"/>
 <part name="R4" library="mf_passives" deviceset="RESISTOR" device="_0603" value="560">
 <attribute name="MPN" value="MF-RES-0603-560"/>
@@
 </part>
 <part name="GND50" library="supply1" deviceset="GND" device=""/>
-<part name="D8" library="mf_leds" deviceset="LED_SINGLE" device="-0603-RED" value="MF-LED-0603-RED"/>
-<part name="D9" library="mf_leds" deviceset="LED_SINGLE" device="-0603-RED" value="MF-LED-0603-RED"/>
-<part name="D10" library="mf_leds" deviceset="LED_SINGLE" device="-0603-GREEN" value="MF-LED-0603-GREEN"/>
+<part name="LED1" library="mf_leds" deviceset="LED_SINGLE" device="-0603-RED" value="MF-LED-0603-RED"/>
+<part name="LED2" library="mf_leds" deviceset="LED_SINGLE" device="-0603-RED" value="MF-LED-0603-RED"/>
+<part name="LED3" library="mf_leds" deviceset="LED_SINGLE" device="-0603-GREEN" value="MF-LED-0603-GREEN"/>
 <part name="GND51" library="supply1" deviceset="GND" device=""/>
 <part name="R33" library="mf_passives" deviceset="RESISTOR" device="_0603" value="1k">
@@
 </part>
 <part name="GND12" library="supply1" deviceset="GND" device=""/>
+<part name="GND13" library="supply1" deviceset="GND" device=""/>
+<part name="R13" library="mf_passives" deviceset="RESISTOR" device="_0603" value="0">
+<attribute name="MPN" value="MF-RES-0603-0"/>
+</part>
+<part name="D1" library="mf_discrete_semiconductor" deviceset="DIODES" device="_SOD-123" technology="_BAT42" value="MF-DIO-SOD123-BAT42"/>
+<part name="D8" library="mf_discrete_semiconductor" deviceset="DIODES" device="_SOD-123" technology="_BAT42" value="MF-DIO-SOD123-BAT42"/>
+<part name="U$2" library="joule_shield" deviceset="V5P0V" device=""/>
 </parts>
 <sheets>
@@
 <instance part="U$58" gate="G$1" x="-10.16" y="172.72"/>
 <instance part="GND12" gate="1" x="-25.4" y="-35.56"/>
+<instance part="GND13" gate="1" x="10.16" y="15.24"/>
+<instance part="R13" gate="G$1" x="10.16" y="25.4"/>
 </instances>
 <busses>
@@
 <junction x="10.16" y="-30.48"/>
 </segment>
+<segment>
+<pinref part="R13" gate="G$1" pin="P$2"/>
+<pinref part="GND13" gate="1" pin="GND"/>
+<wire x1="10.16" y1="20.32" x2="10.16" y2="17.78" width="0.1524" layer="91"/>
+</segment>
 </net>
 <net name="VDD3" class="0">
@@
 <wire x1="81.28" y1="109.22" x2="109.22" y2="109.22" width="0.1524" layer="91"/>
 <label x="93.98" y="109.22" size="1.778" layer="95"/>
+</segment>
+</net>
+<net name="N$10" class="0">
+<segment>
+<pinref part="J6" gate="G$1" pin="USB2_ID_PMIC"/>
+<wire x1="20.32" y1="40.64" x2="10.16" y2="40.64" width="0.1524" layer="91"/>
+<wire x1="10.16" y1="40.64" x2="10.16" y2="30.48" width="0.1524" layer="91"/>
+<pinref part="R13" gate="G$1" pin="P$1"/>
 </segment>
 </net>
@@
 <instance part="GND4" gate="1" x="33.02" y="40.64"/>
 <instance part="R3" gate="G$1" x="45.72" y="35.56" rot="R270"/>
-<instance part="D1" gate="G$1" x="10.16" y="33.02" rot="R270"/>
+<instance part="SYS" gate="G$1" x="10.16" y="33.02" rot="R270"/>
 <instance part="R4" gate="G$1" x="10.16" y="43.18"/>
 <instance part="R5" gate="G$1" x="-2.54" y="20.32"/>
@@
 <net name="N$1" class="0">
 <segment>
-<pinref part="D1" gate="G$1" pin="ANODE"/>
+<pinref part="SYS" gate="G$1" pin="ANODE"/>
 <pinref part="R4" gate="G$1" pin="P$2"/>
 <wire x1="10.16" y1="38.1" x2="10.16" y2="35.56" width="0.1524" layer="91"/>
@@
 <net name="N$6" class="0">
 <segment>
-<pinref part="D1" gate="G$1" pin="CATHODE"/>
+<pinref part="SYS" gate="G$1" pin="CATHODE"/>
 <wire x1="10.16" y1="30.48" x2="10.16" y2="22.86" width="0.1524" layer="91"/>
 <pinref part="U1" gate="G$1" pin="/PG"/>
@@
 <attribute name="POPULATE" x="17.78" y="96.52" size="1.778" layer="96" rot="R90" display="off"/>
 </instance>
-<instance part="FB3" gate="G$1" x="30.48" y="106.68">
-<attribute name="DPN" x="30.48" y="106.68" size="1.778" layer="96" display="off"/>
-<attribute name="MF" x="30.48" y="106.68" size="1.778" layer="96" display="off"/>
-<attribute name="MPN" x="30.48" y="106.68" size="1.778" layer="96" display="off"/>
-<attribute name="POPULATE" x="30.48" y="106.68" size="1.778" layer="96" display="off"/>
+<instance part="FB3" gate="G$1" x="27.94" y="121.92">
+<attribute name="DPN" x="27.94" y="121.92" size="1.778" layer="96" display="off"/>
+<attribute name="MF" x="27.94" y="121.92" size="1.778" layer="96" display="off"/>
+<attribute name="MPN" x="27.94" y="121.92" size="1.778" layer="96" display="off"/>
+<attribute name="POPULATE" x="27.94" y="121.92" size="1.778" layer="96" display="off"/>
 </instance>
 <instance part="C38" gate="G$1" x="43.18" y="99.06"/>
@@
 <instance part="R28" gate="G$1" x="48.26" y="68.58" rot="R90"/>
 <instance part="R29" gate="G$1" x="55.88" y="66.04" rot="R90"/>
+<instance part="D1" gate="G$1" x="43.18" y="116.84" rot="R270"/>
+<instance part="D8" gate="G$1" x="50.8" y="116.84" rot="R270"/>
+<instance part="U$2" gate="G$1" x="50.8" y="127"/>
 </instances>
 <busses>
@@
 <pinref part="D4" gate="G$1" pin="P$2"/>
 <pinref part="FB3" gate="G$1" pin="P$1"/>
-<wire x1="17.78" y1="106.68" x2="20.32" y2="106.68" width="0.1524" layer="91"/>
+<wire x1="17.78" y1="106.68" x2="17.78" y2="121.92" width="0.1524" layer="91"/>
 <pinref part="J1" gate="G$1" pin="5V"/>
 <wire x1="5.08" y1="71.12" x2="7.62" y2="71.12" width="0.1524" layer="91"/>
@@
 <net name="N$49" class="0">
 <segment>
-<pinref part="FB3" gate="G$1" pin="P$2"/>
-<wire x1="40.64" y1="106.68" x2="43.18" y2="106.68" width="0.1524" layer="91"/>
 <pinref part="C38" gate="G$1" pin="P$1"/>
 <wire x1="43.18" y1="106.68" x2="43.18" y2="101.6" width="0.1524" layer="91"/>
@@
 <wire x1="43.18" y1="106.68" x2="50.8" y2="106.68" width="0.1524" layer="91"/>
 <wire x1="50.8" y1="106.68" x2="50.8" y2="73.66" width="0.1524" layer="91"/>
+<pinref part="D1" gate="G$1" pin="CATHODE"/>
+<wire x1="43.18" y1="114.3" x2="43.18" y2="106.68" width="0.1524" layer="91"/>
 <junction x="43.18" y="106.68"/>
+<pinref part="D8" gate="G$1" pin="CATHODE"/>
+<wire x1="50.8" y1="114.3" x2="50.8" y2="106.68" width="0.1524" layer="91"/>
+<junction x="50.8" y="106.68"/>
 </segment>
 </net>
@@
 <pinref part="J1" gate="G$1" pin="D-"/>
 <wire x1="43.18" y1="68.58" x2="5.08" y2="68.58" width="0.1524" layer="91"/>
+</segment>
+</net>
+<net name="N$16" class="0">
+<segment>
+<pinref part="FB3" gate="G$1" pin="P$2"/>
+<wire x1="38.1" y1="121.92" x2="43.18" y2="121.92" width="0.1524" layer="91"/>
+<pinref part="D1" gate="G$1" pin="ANODE"/>
+<wire x1="43.18" y1="121.92" x2="43.18" y2="119.38" width="0.1524" layer="91"/>
+</segment>
+</net>
+<net name="V5P0V" class="0">
+<segment>
+<pinref part="U$2" gate="G$1" pin="V5P0V"/>
+<pinref part="D8" gate="G$1" pin="ANODE"/>
+<wire x1="50.8" y1="127" x2="50.8" y2="119.38" width="0.1524" layer="91"/>
 </segment>
 </net>
@@
 </plain>
 <instances>
-<instance part="D8" gate="G$1" x="50.8" y="50.8" rot="R270"/>
-<instance part="D9" gate="G$1" x="68.58" y="50.8" rot="R270"/>
-<instance part="D10" gate="G$1" x="91.44" y="50.8" rot="R270"/>
+<instance part="LED1" gate="G$1" x="50.8" y="50.8" rot="R270"/>
+<instance part="LED2" gate="G$1" x="68.58" y="50.8" rot="R270"/>
+<instance part="LED3" gate="G$1" x="91.44" y="50.8" rot="R270"/>
 <instance part="GND51" gate="1" x="78.74" y="-20.32"/>
 <instance part="R33" gate="G$1" x="38.1" y="27.94" rot="R180"/>
@@
 <segment>
 <pinref part="R39" gate="G$1" pin="P$2"/>
-<pinref part="D10" gate="G$1" pin="ANODE"/>
+<pinref part="LED3" gate="G$1" pin="ANODE"/>
 <wire x1="91.44" y1="58.42" x2="91.44" y2="53.34" width="0.1524" layer="91"/>
 </segment>
@@
 <segment>
 <pinref part="R38" gate="G$1" pin="P$2"/>
-<pinref part="D9" gate="G$1" pin="ANODE"/>
+<pinref part="LED2" gate="G$1" pin="ANODE"/>
 <wire x1="68.58" y1="58.42" x2="68.58" y2="53.34" width="0.1524" layer="91"/>
 </segment>
@@
 <segment>
 <pinref part="R37" gate="G$1" pin="P$2"/>
-<pinref part="D8" gate="G$1" pin="ANODE"/>
+<pinref part="LED1" gate="G$1" pin="ANODE"/>
 <wire x1="50.8" y1="58.42" x2="50.8" y2="53.34" width="0.1524" layer="91"/>
 </segment>
@@
 <net name="N$59" class="0">
 <segment>
-<pinref part="D8" gate="G$1" pin="CATHODE"/>
+<pinref part="LED1" gate="G$1" pin="CATHODE"/>
 <wire x1="50.8" y1="48.26" x2="50.8" y2="40.64" width="0.1524" layer="91"/>
 <pinref part="Q1" gate="G$1" pin="D"/>
@@
 <net name="N$60" class="0">
 <segment>
-<pinref part="D9" gate="G$1" pin="CATHODE"/>
+<pinref part="LED2" gate="G$1" pin="CATHODE"/>
 <wire x1="68.58" y1="48.26" x2="68.58" y2="27.94" width="0.1524" layer="91"/>
 <pinref part="Q2" gate="G$1" pin="D"/>
@@
 <net name="N$61" class="0">
 <segment>
-<pinref part="D10" gate="G$1" pin="CATHODE"/>
+<pinref part="LED3" gate="G$1" pin="CATHODE"/>
 <wire x1="91.44" y1="48.26" x2="91.44" y2="12.7" width="0.1524" layer="91"/>
 <pinref part="Q3" gate="G$1" pin="D"/>

Commit message: joule shield checkpoint
Connections:
- net N$28 renamed VDC_JACK
Changed lines of the file:
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@@
 </segment>
 </net>
-<net name="N$28" class="0">
+<net name="VDC_JACK" class="0">
 <segment>
 <pinref part="JD1" gate="G$1" pin="4"/>
@@
 <wire x1="50.8" y1="106.68" x2="48.26" y2="106.68" width="0.1524" layer="91"/>
 <wire x1="48.26" y1="106.68" x2="48.26" y2="81.28" width="0.1524" layer="91"/>
+<label x="40.64" y="99.06" size="1.778" layer="95"/>
 </segment>
 </net>

Commit message: joule shield checkpoint
Connections:
- net PMIC_PWRBTN_N: now also J6.PMIC_PWRBTN_N
Changed lines of the file:
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@@
+</segment>
+</net>
+<net name="PMIC_PWRBTN_N" class="0">
+<segment>
+<pinref part="J6" gate="G$1" pin="PMIC_PWRBTN_N"/>
+<wire x1="81.28" y1="33.02" x2="116.84" y2="33.02" width="0.1524" layer="91"/>
+<label x="101.6" y="33.02" size="1.778" layer="95"/>
 </segment>
 </net>
@@
 <instance part="U$43" gate="G$1" x="180.34" y="73.66"/>
 <instance part="R27" gate="G$1" x="180.34" y="55.88"/>
-<instance part="GND44" gate="1" x="149.86" y="20.32"/>
+<instance part="GND44" gate="1" x="149.86" y="12.7"/>
 <instance part="PWR" gate="G$1" x="17.78" y="124.46"/>
 <instance part="DNX" gate="G$1" x="88.9" y="124.46"/>
@@
 <wire x1="139.7" y1="27.94" x2="149.86" y2="27.94" width="0.1524" layer="91"/>
 <pinref part="GND44" gate="1" pin="GND"/>
-<wire x1="149.86" y1="27.94" x2="149.86" y2="22.86" width="0.1524" layer="91"/>
+<wire x1="149.86" y1="27.94" x2="149.86" y2="15.24" width="0.1524" layer="91"/>
 <pinref part="JFAN" gate="G$1" pin="3"/>
 <wire x1="139.7" y1="35.56" x2="149.86" y2="35.56" width="0.1524" layer="91"/>
