File: hw/pi3_hat/pi3_hat.sch (EAGLE design)
At the start: 17 parts, among them U1 SINGLE-BIT_BUS_TRANSCEIVER, U2 SINGLE-BIT_BUS_TRANSCEIVER, U3 ST1S10, U4 DMMT5401, U5 DMG2305UX

Commit message: rpi3 hat as sent to macrofab
Parts:
- C2: DPN 399-7442-1-ND -> (none); MFG (none) -> MF; MPN (none) -> MF-CAP-1206-10u
- C3: DPN 399-7847-1-ND -> (none); MFG (none) -> TDK; MPN (none) -> C1608X7R1C105K080AC
- C4: DPN 445-3955-1-ND -> (none); MFG (none) -> TDK; MPN (none) -> CGA6P1X7R1C226M250AC
Changed lines of the file:
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@@
 <part name="GND5" library="supply1" deviceset="GND" device=""/>
 <part name="C2" library="rcl" deviceset="C-US" device="C1206" value="10uF 16V">
-<attribute name="DPN" value="399-7442-1-ND"/>
+<attribute name="MFG" value="MF"/>
+<attribute name="MPN" value="MF-CAP-1206-10u"/>
 </part>
 <part name="C3" library="rcl" deviceset="C-US" device="C0603" value="1uF 16V">
-<attribute name="DPN" value="399-7847-1-ND"/>
+<attribute name="MFG" value="TDK"/>
+<attribute name="MPN" value="C1608X7R1C105K080AC"/>
 </part>
 <part name="C4" library="rcl" deviceset="C-US" device="C1210" value="22uF 16V">
-<attribute name="DPN" value="445-3955-1-ND"/>
+<attribute name="MFG" value="TDK"/>
+<attribute name="MPN" value="CGA6P1X7R1C226M250AC"/>
 </part>
 <part name="L1" library="odroid_shield" deviceset="L-US" device="WURTH_74404042033" value="3.3uH">
@@
 <instance part="GND5" gate="1" x="63.5" y="-2.54"/>
 <instance part="C2" gate="G$1" x="15.24" y="33.02">
-<attribute name="DPN" x="15.24" y="33.02" size="1.778" layer="96" display="off"/>
+<attribute name="MFG" x="15.24" y="33.02" size="1.778" layer="96" display="off"/>
+<attribute name="MPN" x="15.24" y="33.02" size="1.778" layer="96" display="off"/>
 </instance>
 <instance part="C3" gate="G$1" x="22.86" y="22.86">
-<attribute name="DPN" x="22.86" y="22.86" size="1.778" layer="96" display="off"/>
+<attribute name="MFG" x="22.86" y="22.86" size="1.778" layer="96" display="off"/>
+<attribute name="MPN" x="22.86" y="22.86" size="1.778" layer="96" display="off"/>
 </instance>
 <instance part="C4" gate="G$1" x="114.3" y="27.94">
-<attribute name="DPN" x="114.3" y="27.94" size="1.778" layer="96" display="off"/>
+<attribute name="MFG" x="114.3" y="27.94" size="1.778" layer="96" display="off"/>
+<attribute name="MPN" x="114.3" y="27.94" size="1.778" layer="96" display="off"/>
 </instance>
 <instance part="L1" gate="G$1" x="93.98" y="35.56" rot="R90">

Commit message: Fix part number on regulator to HSOP-8 package
Parts:
- U3: MPN ST1S40IPUR -> ST1S40IPHR
Changed lines of the file:
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@@
 <attribute name="DPN" value="497-12084-1-ND"/>
 <attribute name="MF" value="STMicroelectronics"/>
-<attribute name="MPN" value="ST1S40IPUR"/>
+<attribute name="MPN" value="ST1S40IPHR"/>
 </part>
 <part name="GND5" library="supply1" deviceset="GND" device=""/>

Commit message: Work on updated pi3 hat
Parts:
- added C10, C9: 10pF, mfpassives:CAPACITOR_NP_0603
- added C11, C12: .1uF, mfpassives:CAPACITOR_NP_0603
- added C13: 1uF, mfpassives:CAPACITOR_NP_0603
- added C5, C8: 22uF 16V, mfpassives:CAPACITOR_NP_1210
- added C6: 10uF 35V, mfpassives:CAPACITOR_NP_1206
- added C7: 1uF 16V, mfpassives:CAPACITOR_NP_0603
- added D1: MF-LED-0603-RED, mfleds:LED_SINGLE-0603-RED
- added D2: MF-LED-0603-GREEN, mfleds:LED_SINGLE-0603-GREEN
- added R5, R7, R8: 220, mfpassives:RESISTOR_0603
- added R6: 120, mfpassives:RESISTOR_0603
- added SWD: JST-ZH6SMT_VERT, controller:JST-ZH6SMT_VERT
- added X1: 8.0MHz, controller:CRYSTALABM3B
- C1: value 0.1uF -> .1uF; device rcl:C-USC0603 -> mfpassives:CAPACITOR_NP_0603; HOUSEPART (none) -> 1; MPN (none) -> MF-CAP-0603-0.1uF
- C2: value 10uF 16V -> 10uF 35V; device rcl:C-USC1206 -> mfpassives:CAPACITOR_NP_1206; MF (none) -> TDK; MFG MF -> (none); MPN MF-CAP-1206-10u -> CGA5L1X7R1V106K160AC
- C3: value 1uF 16V -> .1uF 50V; device rcl:C-USC0603 -> mfpassives:CAPACITOR_NP_0805; HOUSEPART (none) -> 1; MFG TDK -> (none); MPN C1608X7R1C105K080AC -> MF-CAP-0805-0.1uF
- C4: value 22uF 16V -> 1uF; device rcl:C-USC1210 -> mfpassives:CAPACITOR_NP_0603; HOUSEPART (none) -> 1; MFG TDK -> (none); MPN CGA6P1X7R1C226M250AC -> MF-CAP-0603-1uF
- L1: value 3.3uH -> 6.8uH 3.7A; device odroid_shield:L-USWURTH_74404042033 -> pi3_hat:INDUCTORTAIYO_8040; DPN 732-5505-1-ND -> (none); HOUSEPART (none) -> 0; MF (none) -> TAIYO YUDEN; MPN (none) -> NR8040T6R8N; POPULATE (none) -> 1
- R1: value 105k 1% -> 27k 1%; device rcl:R-US_R0603 -> mfpassives:RESISTOR_0603; DPN P105KHCT-ND -> (none)
- R2: value 20k 1% -> 5.1k 1%; device rcl:R-US_R0603 -> mfpassives:RESISTOR_0603; DPN P20.0KHCT-ND -> (none)
- U1: value SINGLE-BIT_BUS_TRANSCEIVER -> MAX13431E; device odroid_shield:SINGLE-BIT_BUS_TRANSCEIVER -> controller:MAX13431E; DPN 296-16843-1-ND -> (none); MF (none) -> Maxim; MPN (none) -> MAX13431EETB+T; POPULATE (none) -> 1
- U2: value SINGLE-BIT_BUS_TRANSCEIVER -> RT829910L_DFN; device odroid_shield:SINGLE-BIT_BUS_TRANSCEIVER -> pi3_hat:RT829910L_DFN; DPN 296-16843-1-ND -> (none)
- U3: value ST1S10 -> STM32F051X6UFQFPN32; device odroid_shield:ST1S10 -> pi3_hat:STM32F051X6UFQFPN32; DPN 497-12084-1-ND -> (none); MF STMicroelectronics -> (none); MPN ST1S40IPHR -> (none)
Connections:
- net N$7 renamed +18V
- removed net N$10: L1.1, U3.SW
- removed net PI_RX_5V: JD1.2, U1.A
- removed net PI_TX_5V: JD1.3, U2.B
- removed net VCCIO: C1.1, JP1.1, U1.VCCB, U2.DIR, U2.VCCA
- new net +3V3: C1.P$1, C12.P$1, C13.P$1, C4.P$1, JP1.1, R7.P$2, R8.P$2, SWD.6, U1.VCC, U1.VL, U3.VDD, U3.VDDA
- new net 485_DIR: U1.DE, U1.RE/, U3.PA1/USART2_RTS/TIM2_CH2/ADC1
- new net 485_RX: U1.RO, U3.PA3/USART2_RX/TIM2_CH4/TIM15_CH2
- new net 485_TX: U1.DI, U3.PA2/USART2_TX/TIM2_CH3/TIM15_CH1/ADC2
- new net N$12: SWD.5, U3.PA14/SWCLK
- new net N$15: D1.ANODE, R7.P$1
- new net N$16: D2.ANODE, R8.P$1
- new net N$17: D1.CATHODE, U3.PB3/SPI1_SCK/TIM2_CH2
- new net N$18: D2.CATHODE, U3.PB4/SPI1_MISO/TIM3_CH1
- new net N$35: C9.P$1, U3.PF1-OSC_OUT, X1.P$1
- new net N$36: C10.P$1, U3.PF0-OSC_IN, X1.P$2
- new net N$8: C3.P$1, U2.BOOT
- new net NRST: C11.P$1, SWD.2, U3.NRST
- new net PI_RX_3V: JP1.10, U3.PA9/USART1_TX/TIM1_CH2
- new net PI_TX_3V: JP1.8, U3.PA10/USART1_RX/TIM1_CH3
- new net POSTFUSE: C2.P$1, C6.P$1, F1.2, U2.VIN
- new net RS485_N: JD1.3, R6.P$2, U1.B
- new net RS485_P: JD1.2, R6.P$1, U1.A
- new net SW: C3.P$2, L1.P$1, U2.SW
- net +5V: no longer U1.DIR, U1.VCCA, U2.VCCB
- net GND: now also C1.P$2, C10.P$2, C11.P$2, C12.P$2, C13.P$2, C2.P$2, C4.P$2, C5.P$2, C6.P$2, C7.P$2, C8.P$2, C9.P$2, R2.P$2, R5.P$2, SWD.4, U3.VSS, X1.P$3; no longer C1.2, C2.2, C3.2, C4.2, R2.1, U3.AGND, U3.PAD, U3.PGND, U3.SYNC
- net N$11: now also R1.P$2, R2.P$1, U2.FB; no longer C2.1, C3.1, F1.2, U3.EN, U3.VIN_A, U3.VIN_SW
- net N$13: now also SWD.3, U3.PA13/SWDIO; no longer R1.1, R2.2, U3.FB
- net N$2: now also C7.P$1, U2.VCC; no longer JP1.10, U1.B
- net N$4: now also R5.P$1, U3.BOOT0; no longer JP1.8, U2.A
- net REGOUT: now also C5.P$1, C8.P$1, L1.P$2, R1.P$1; no longer C4.1, L1.2, R1.2
Other:
- moved on the sheet: R1, R2

Commit message: Nominally complete pi3 hat
Parts:
- added R9: 220, mfpassives:RESISTOR_0603
- C1, C11, C12: value .1uF -> .1uF 50V; device mfpassives:CAPACITOR_NP_0603 -> mfpassives:CAPACITOR_NP_0805; MPN MF-CAP-0603-0.1uF -> MF-CAP-0805-0.1uF
- C7: value 1uF 16V -> 1uF
- F1: MPN (none) -> MFU0603FF04000P100; POPULATE (none) -> 1
- JD1: MF (none) -> JST; MPN (none) -> S4B-XH-SM4-TB(LF)(SN); POPULATE (none) -> 1
- JP1: POPULATE (none) -> 0
- R1: value 27k 1% -> 53.6k 1%; MF (none) -> Panasonic; MPN (none) -> ERJ-3EKF5362V
- R2: value 5.1k 1% -> 10k 1%; MF (none) -> Panasonic; MPN (none) -> ERJ-3EKF1002V
- R3: device rcl:R-US_R0603 -> mfpassives:RESISTOR_0603; DPN MCT0603-10.0K-CFCT-ND -> (none); MF (none) -> Panasonic; MPN (none) -> ERJ-3EKF1002V
- R4: value 47k 1% -> 53.6k 1%; device rcl:R-US_R0603 -> mfpassives:RESISTOR_0603; DPN P47.0KHCT-ND -> (none); MF (none) -> Panasonic; MPN (none) -> ERJ-3EKF5362V
- R6: value 120 -> 220; MPN (none) -> MF-RES-0603-220
- U2: POPULATE (none) -> 1
- U3: MF (none) -> STMicroelectronics; MPN (none) -> STM32F051K6U6; POPULATE (none) -> 1
- U4: MF (none) -> Didoes Incorporated; MPN (none) -> DMMT5401-7-F; POPULATE (none) -> 1
- U5: MF (none) -> Diodes Incorporated; MPN (none) -> DMG2305UX-13; POPULATE (none) -> 1
Connections:
- net GND: now also R3.P$2, R4.P$2; no longer R3.1, R4.1
- net N$1: now also R3.P$1; no longer R3.2
- net N$5: now also R4.P$1; no longer R4.2
- net RS485_N: now also JD1.2, R6.P$1, R9.P$1; no longer JD1.3, R6.P$2
- net RS485_P: now also JD1.3, R6.P$2, R9.P$2; no longer JD1.2, R6.P$1
Other:
- moved on the sheet: R3, R4, R6
