File: hw/pi3_hat/pcb/pi3_hat.brd (EAGLE design)
At the start: 56.5 x 28.5 mm, 35 parts, among them U1 MAX13431E, U2 RT829910L_DFN, U3 STM32F051X6UFQFPN32, U4 DMMT5401, U5 DMG2305UX, X1 8.0MHz

Commit message: Make r3 of pi3 hat
Parts:
- added R10: 53.6k 1%, mfpassives:R0603
- moved C3 0.30 mm to (50.8, 24.5)
Connections:
- new net N$7: R10.P$2, U2.3
- net POSTFUSE: now also R10.P$1
Routing:
- net POSTFUSE: track 4.12 -> 10.8 mm
- net N$7: track 0.00 -> 5.24 mm
Other:
- board text added: "mjmech pi3hat r3"
- board text removed: "mjmech pi3hat r2"
Changed lines of the file:
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@@
 <text x="56" y="13" size="1" layer="21" ratio="10" rot="R180">jjp@pobox.com</text>
 <text x="56" y="11.5" size="1" layer="21" ratio="10" rot="R180">(c) 2019</text>
-<text x="56" y="10" size="1" layer="21" ratio="10" rot="R180">mjmech pi3hat r2</text>
+<text x="56" y="10" size="1" layer="21" ratio="10" rot="R180">mjmech pi3hat r3</text>
 </plain>
 <attributes>
@@
 <attribute name="NAME" x="52.9" y="22.8" size="0.6" layer="25" font="vector" ratio="10"/>
 </element>
-<element name="C3" library="mfpassives" package="C0805" value=".1uF 50V" x="50.5" y="24.5" smashed="yes" rot="R90">
-<attribute name="HOUSEPART" value="1" x="50.5" y="24.5" size="1.778" layer="27" rot="R90" display="off"/>
-<attribute name="TOLERANCE" value="" x="50.5" y="24.5" size="1.778" layer="27" rot="R90" display="off"/>
-<attribute name="MPN" value="MF-CAP-0805-0.1uF" x="50.5" y="24.5" size="1.778" layer="27" rot="R90" display="off"/>
-<attribute name="POPULATE" value="1" x="50.5" y="24.5" size="1.778" layer="27" rot="R90" display="off"/>
-<attribute name="DIELECTRIC" value="" x="50.5" y="24.5" size="1.778" layer="27" rot="R90" display="off"/>
-<attribute name="VOLTAGE" value="" x="50.5" y="24.5" size="1.778" layer="27" rot="R90" display="off"/>
-<attribute name="URL" value="" x="50.5" y="24.5" size="1.778" layer="27" rot="R90" display="off"/>
-<attribute name="NAME" x="50.8" y="26.5" size="0.6" layer="25" font="vector" ratio="10"/>
+<element name="C3" library="mfpassives" package="C0805" value=".1uF 50V" x="50.8" y="24.5" smashed="yes" rot="R90">
+<attribute name="HOUSEPART" value="1" x="50.8" y="24.5" size="1.778" layer="27" rot="R90" display="off"/>
+<attribute name="TOLERANCE" value="" x="50.8" y="24.5" size="1.778" layer="27" rot="R90" display="off"/>
+<attribute name="MPN" value="MF-CAP-0805-0.1uF" x="50.8" y="24.5" size="1.778" layer="27" rot="R90" display="off"/>
+<attribute name="POPULATE" value="1" x="50.8" y="24.5" size="1.778" layer="27" rot="R90" display="off"/>
+<attribute name="DIELECTRIC" value="" x="50.8" y="24.5" size="1.778" layer="27" rot="R90" display="off"/>
+<attribute name="VOLTAGE" value="" x="50.8" y="24.5" size="1.778" layer="27" rot="R90" display="off"/>
+<attribute name="URL" value="" x="50.8" y="24.5" size="1.778" layer="27" rot="R90" display="off"/>
+<attribute name="NAME" x="51.1" y="26.5" size="0.6" layer="25" font="vector" ratio="10"/>
 </element>
 <element name="R1" library="mfpassives" package="R0603" value="53.6k 1%" x="53.3" y="20.3" smashed="yes" rot="R180">
@@
 <attribute name="WATTAGE" value="" x="22.6" y="24.85" size="1.778" layer="28" rot="MR0" display="off"/>
 <attribute name="NAME" x="21" y="24.45" size="0.6" layer="26" font="vector" ratio="10" rot="MR0"/>
+</element>
+<element name="R10" library="mfpassives" package="R0603" value="53.6k 1%" x="52.9" y="25.1" smashed="yes" rot="R270">
+<attribute name="HOUSEPART" value="" x="52.9" y="25.1" size="1.778" layer="27" rot="R270" display="off"/>
+<attribute name="TOLERANCE" value="" x="52.9" y="25.1" size="1.778" layer="27" rot="R270" display="off"/>
+<attribute name="MPN" value="ERJ-3EKF5362V" x="52.9" y="25.1" size="1.778" layer="27" rot="R270" display="off"/>
+<attribute name="POPULATE" value="1" x="52.9" y="25.1" size="1.778" layer="27" rot="R270" display="off"/>
+<attribute name="VOLTAGE" value="" x="52.9" y="25.1" size="1.778" layer="27" rot="R270" display="off"/>
+<attribute name="MF" value="Panasonic" x="52.9" y="25.1" size="1.778" layer="27" rot="R270" display="off"/>
+<attribute name="URL" value="" x="52.9" y="25.1" size="1.778" layer="27" rot="R270" display="off"/>
+<attribute name="WATTAGE" value="" x="52.9" y="25.1" size="1.778" layer="27" rot="R270" display="off"/>
+<attribute name="NAME" x="54" y="26.5" size="0.6" layer="25" font="vector" ratio="10" rot="R270"/>
 </element>
 </elements>
@@
 <vertex x="46.5" y="18.2"/>
 </polygon>
-<wire x1="50.5" y1="25.45" x2="50.7" y2="24.5" width="0.254" layer="1"/>
+<wire x1="50.8" y1="25.45" x2="50.7" y2="24.5" width="0.254" layer="1"/>
 <via x="50.7" y="24.5" extent="1-16" drill="0.4"/>
 <wire x1="50.7" y1="24.5" x2="50.7" y2="19.3" width="0.254" layer="16"/>
@@
 <vertex x="48.9" y="23.6"/>
 </polygon>
+<contactref element="R10" pad="P$1"/>
+<wire x1="49.8" y1="26" x2="52.8" y2="26" width="0.127" layer="1"/>
+<wire x1="49.8" y1="24.4" x2="49.8" y2="26" width="0.127" layer="1"/>
+<wire x1="49" y1="23.6" x2="49.8" y2="24.4" width="0.127" layer="1"/>
+<wire x1="52.8" y1="26" x2="52.9" y2="25.85" width="0.127" layer="1"/>
+<wire x1="49" y1="23.6" x2="48.3" y2="23.45" width="0.127" layer="1"/>
 </signal>
 <signal name="N$8">
 <contactref element="U2" pad="5"/>
 <contactref element="C3" pad="P$1"/>
-<wire x1="50.5" y1="23.55" x2="51.4" y2="22.65" width="0.3048" layer="1"/>
+<wire x1="50.8" y1="23.55" x2="51.4" y2="22.65" width="0.3048" layer="1"/>
 <wire x1="51.4" y1="22.65" x2="51.4" y2="22.6" width="0.3048" layer="1"/>
 <wire x1="51.4" y1="22.6" x2="51.425" y2="22.575" width="0.254" layer="1"/>
@@
 <wire x1="20.75" y1="2.9" x2="20.75" y2="4.65" width="0.254" layer="1"/>
 </signal>
+<signal name="N$7">
+<contactref element="R10" pad="P$2"/>
+<contactref element="U2" pad="3"/>
+<wire x1="53.2" y1="21" x2="51.425" y2="21" width="0.127" layer="1"/>
+<wire x1="53.2" y1="24" x2="53.2" y2="21" width="0.127" layer="1"/>
+<wire x1="53" y1="24.2" x2="53.2" y2="24" width="0.127" layer="1"/>
+<wire x1="53" y1="24.2" x2="52.9" y2="24.35" width="0.127" layer="1"/>
+</signal>
 </signals>
