File: hw/pi3_hat/pcb/pi3_hat.sch (EAGLE design)
At the start: 35 parts, among them U1 MAX13431E, U2 RT829910L_DFN, U3 STM32F051X6UFQFPN32, U4 DMMT5401, U5 DMG2305UX, X1 8.0MHz

Commit message: Make r3 of pi3 hat
Parts:
- added R10: 53.6k 1%, mfpassives:RESISTOR_0603
Connections:
- new net N$7: R10.P$2, U2.EN
- net POSTFUSE: now also R10.P$1
Changed lines of the file:
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@@
 <attribute name="MPN" value="MF-RES-0603-220"/>
+</part>
+<part name="R10" library="mfpassives" deviceset="RESISTOR" device="_0603" value="53.6k 1%">
+<attribute name="MF" value="Panasonic"/>
+<attribute name="MPN" value="ERJ-3EKF5362V"/>
 </part>
 </parts>
@@
 <instance part="R6" gate="G$1" x="246.38" y="157.48" rot="R180"/>
 <instance part="R9" gate="G$1" x="254" y="157.48" rot="R180"/>
+<instance part="R10" gate="G$1" x="33.02" y="35.56">
+<attribute name="MF" x="33.02" y="35.56" size="1.778" layer="96" display="off"/>
+</instance>
 </instances>
 <busses>
@@
 <wire x1="10.16" y1="35.56" x2="10.16" y2="33.02" width="0.1524" layer="91"/>
 <pinref part="C2" gate="G$1" pin="P$1"/>
-<wire x1="10.16" y1="35.56" x2="17.78" y2="35.56" width="0.1524" layer="91"/>
-<wire x1="17.78" y1="35.56" x2="17.78" y2="33.02" width="0.1524" layer="91"/>
+<wire x1="10.16" y1="35.56" x2="17.78" y2="40.64" width="0.1524" layer="91"/>
+<wire x1="17.78" y1="40.64" x2="17.78" y2="33.02" width="0.1524" layer="91"/>
 <junction x="10.16" y="35.56"/>
 <pinref part="U2" gate="G$1" pin="VIN"/>
 <wire x1="45.72" y1="38.1" x2="48.26" y2="38.1" width="0.1524" layer="91"/>
-<wire x1="45.72" y1="35.56" x2="45.72" y2="38.1" width="0.1524" layer="91"/>
-<wire x1="17.78" y1="35.56" x2="45.72" y2="35.56" width="0.1524" layer="91"/>
-<junction x="17.78" y="35.56"/>
+<wire x1="45.72" y1="40.64" x2="45.72" y2="38.1" width="0.1524" layer="91"/>
+<wire x1="17.78" y1="40.64" x2="33.02" y2="40.64" width="0.1524" layer="91"/>
+<junction x="17.78" y="40.64"/>
 <label x="12.7" y="35.56" size="1.778" layer="95"/>
+<pinref part="R10" gate="G$1" pin="P$1"/>
+<wire x1="33.02" y1="40.64" x2="45.72" y2="40.64" width="0.1524" layer="91"/>
+<junction x="33.02" y="40.64"/>
 </segment>
 </net>
@@
 </segment>
 </net>
+<net name="N$7" class="0">
+<segment>
+<pinref part="R10" gate="G$1" pin="P$2"/>
+<pinref part="U2" gate="G$1" pin="EN"/>
+<wire x1="33.02" y1="30.48" x2="48.26" y2="30.48" width="0.1524" layer="91"/>
+</segment>
+</net>
