File: hw/aeg_driver/aeg_driver.sch (EAGLE design)
At the start: 48 parts, among them J1 JST-ZH6SMT_VERT, J2 XT30XT30PW_MALE, U1 MAX150628TDFN, U2 TCAN334GSOT23, U3 STM32G474CEU6, U4 MC33926, U5 MC33926

Commit message: aeg_driver: Route drive, renumber, resize silks, rough silk place
Parts:
- removed C22, C23, C24: 10uF 50V, mfpassives:CAPACITOR_NP_1206
- removed C25: 100uF, aeg_driver:CPOL-USFT_D
- removed JP1, JP4: (no value), pinhead:PINHD-1X2
- removed R13: 18k, mfpassives:RESISTOR_0603
- removed R7: 560, mfpassives:RESISTOR_0603
- removed U8: (no value), mfdiscrete:N-CHANNEL_FET_SOT-23-3
- added C17, C18, C19: 10uF 50V, mfpassives:CAPACITOR_NP_1206
- added C20: 0.1uF 50V, mfpassives:CAPACITOR_NP_0402
- added J5: XT30XT30PW_MALE, controller:XT30XT30PW_MALE
- added J6: JST-ZH6SMT_VERT, precharge:JST-ZH6SMT_VERT
- added R5: 18k, mfpassives:RESISTOR_0603
- added R6: 560, mfpassives:RESISTOR_0603
- added U6: MC33926, gimbal:MC33926
- C1: value 0.1uF -> 100uF; device mfpassives:CAPACITOR_NP_0402 -> aeg_driver:CPOL-USFT_D; HOUSEPART 1 -> (none); MF (none) -> PANASONIC; MPN MF-CAP-0402-0.1uF -> EEE-FT1V101AP; POPULATE (none) -> 1
- C10: value 0.1uF -> 10uF 35V; device mfpassives:CAPACITOR_NP_0402 -> mfpassives:CAPACITOR_NP_1206; HOUSEPART 1 -> (none); MF (none) -> TDK; MPN MF-CAP-0402-0.1uF -> CGA5L1X7R1V106K160AC
- C11: HOUSEPART YES -> 1
- C12: HOUSEPART 1 -> YES
- C13: value 0.1uF -> 10uF 50V; device mfpassives:CAPACITOR_NP_0402 -> mfpassives:CAPACITOR_NP_1206; HOUSEPART 1 -> (none); MF (none) -> TDK; MPN MF-CAP-0402-0.1uF -> C3216X7R1H106K160AE
- C14: value 1uF -> 10uF 50V; device mfpassives:CAPACITOR_NP_0402 -> mfpassives:CAPACITOR_NP_1206; HOUSEPART 1 -> (none); MF (none) -> TDK; MPN MF-CAP-0402-1uF -> C3216X7R1H106K160AE
- C15: value 10uF 35V -> 10uF 50V; MPN CGA5L1X7R1V106K160AC -> C3216X7R1H106K160AE
- C2: value 0.1uF 50V -> 1uF 50V; device mfpassives:CAPACITOR_NP_0402 -> mfpassives:CAPACITOR_NP_0603; MF Walsin -> SAMSUNG; MPN 0402B104K500CT -> CL10A105KB8NNNC
- C3: value 0.1uF -> 1uF 50V; device mfpassives:CAPACITOR_NP_0402 -> mfpassives:CAPACITOR_NP_0603; HOUSEPART 1 -> (none); MF (none) -> SAMSUNG; MPN MF-CAP-0402-0.1uF -> CL10A105KB8NNNC
- C4: value 10uF 50V -> 10uF 35V; MPN C3216X7R1H106K160AE -> CGA5L1X7R1V106K160AC
- C5, C6: value 10uF 50V -> 0.1uF; device mfpassives:CAPACITOR_NP_1206 -> mfpassives:CAPACITOR_NP_0402; HOUSEPART (none) -> 1; MF TDK -> (none); MPN C3216X7R1H106K160AE -> MF-CAP-0402-0.1uF
- C7: value 10uF 35V -> 1uF; device mfpassives:CAPACITOR_NP_1206 -> mfpassives:CAPACITOR_NP_0402; HOUSEPART (none) -> 1; MF TDK -> (none); MPN CGA5L1X7R1V106K160AC -> MF-CAP-0402-1uF
- C8, C9: value 1uF 50V -> 0.1uF; device mfpassives:CAPACITOR_NP_0603 -> mfpassives:CAPACITOR_NP_0402; HOUSEPART (none) -> 1; MF SAMSUNG -> (none); MPN CL10A105KB8NNNC -> MF-CAP-0402-0.1uF
- J1: value JST-ZH6SMT_VERT -> (none); device precharge:JST-ZH6SMT_VERT -> pinhead:PINHD-1X2; MF JST -> (none); MPN B6B-ZR-SM4-TF(LF)(SN) -> (none); POPULATE 1 -> (none)
- J2: value XT30XT30PW_MALE -> (none); device controller:XT30XT30PW_MALE -> pinhead:PINHD-1X2; POPULATE 0 -> (none)
- R1: value 18k -> 220; MPN MF-RES-0603-18K -> MF-RES-0603-220
- R2: value 560 -> 220; MPN MF-RES-0603-560 -> MF-RES-0603-220
- R3: value 220 -> 18k; MPN MF-RES-0603-220 -> MF-RES-0603-18K
- R4: value 220 -> 560; MPN MF-RES-0603-220 -> MF-RES-0603-560
- U1: value MAX150628TDFN -> (none); device precharge:MAX150628TDFN -> mfdiscrete:N-CHANNEL_FET_SOT-23-3; HOUSEPART (none) -> YES; MF MAXIM -> (none); MPN MAX15062AATA+T -> MF-DSC-SOT233-BSS138
- U2: value TCAN334GSOT23 -> MAX150628TDFN; device controller:TCAN334GSOT23 -> precharge:MAX150628TDFN; MF TI -> MAXIM; MPN TCAN334GDCNT -> MAX15062AATA+T
- U4: value MC33926 -> TCAN334GSOT23; device gimbal:MC33926 -> controller:TCAN334GSOT23; MF Freescale -> TI; MPN MC33926PNBR2 -> TCAN334GDCNT
- renumbered C21 to C16, JP2 to J4, JP3 to J3
Connections:
- net AEG_D1: now also U6.D1; no longer U5.D1
- net AEG_FB: now also R6.P$2, U6.FB; no longer R2.P$2, U5.FB
- net AEG_OUT: now also U6.OUT1; no longer U5.OUT1
- net AEG_PWM: now also U6.IN1; no longer U5.IN1
- net AEG_SF: now also R5.P$1, U6.SF/; no longer R1.P$1, U5.SF/
- net CAN_N: now also U4.CANL; no longer U2.CANL
- net CAN_P: now also U4.CANH; no longer U2.CANH
- net CAN_RX: now also U4.RXD; no longer U2.RXD
- net CAN_TX: now also U4.TXD; no longer U2.TXD
- net GLOBAL_EN: now also U6.EN; no longer U4.EN
- net GND: now also C1.-, C17.P$2, C18.P$2, C19.P$2, C2.P$2, J5.2, J6.4, R4.P$1, R6.P$1, U1.SOURCE, U4.GND, U4.SHDN, U4.STB, U6.AGND, U6.PAD, U6.PGND; no longer C1.P$2, C22.P$2, C23.P$2, C24.P$2, C25.-, J1.4, J2.2, R2.P$1, R7.P$1, U1.GND, U2.SHDN, U2.STB, U4.AGND, U4.PAD, U4.PGND, U8.SOURCE
- net LASER_EN: now also U1.GATE; no longer U8.GATE
- net LOADER_D1: now also U5.D1; no longer U4.D1
- net LOADER_FB: now also R4.P$2, U5.FB; no longer R7.P$2, U4.FB
- net LOADER_OUT1: now also J2.1, U5.OUT1; no longer JP1.1, U4.OUT1
- net LOADER_OUT2: now also J2.2, U5.OUT2; no longer JP1.2, U4.OUT2
- net LOADER_PWM1: now also U5.IN1; no longer U4.IN1
- net LOADER_PWM2: now also U5.IN2; no longer U4.IN2
- net LOADER_SF: now also R3.P$1, U5.SF/; no longer R13.P$1, U4.SF/
- net LX: now also U2.LX; no longer U1.LX
- net MISC_OUT: now also U6.OUT2; no longer U5.OUT2
- net MISC_PWM: now also U6.IN2; no longer U5.IN2
- net N$1: now also C20.P$2, U6.CCP; no longer C2.P$2, U5.CCP
- net N$13: now also C3.P$1, U2.VCC; no longer C9.P$1, U1.VCC
- net N$2: now also J1.2, U1.DRAIN; no longer JP4.2, U8.DRAIN
- net N$3: now also J5.1; no longer J2.1
- net N$39: now also R1.P$1; no longer R3.P$1
- net N$40: now also R2.P$1; no longer R4.P$1
- net N$5: now also U5.CCP; no longer U4.CCP
- net NRST: now also C5.P$1, J6.2; no longer C3.P$1, J1.2
- net SWCLK: now also J6.5; no longer J1.5
- net SWDIO: now also J6.3; no longer J1.3
- net V+: now also C1.+, C13.P$1, C14.P$1, C15.P$1, C17.P$1, C18.P$1, C19.P$1, C20.P$1, U2.EN, U2.VIN, U6.VPWR; no longer C22.P$1, C23.P$1, C24.P$1, C25.+, C4.P$1, C5.P$1, C6.P$1, C8.P$1, U1.EN, U1.VIN, U4.VPWR
- net VCC: now also C4.P$1, C6.P$1, C8.P$1, C9.P$1, J1.1, J6.6, R2.P$2, R5.P$2, U2.FB, U4.VCC, U6.D2/, U6.SLEW; no longer C1.P$1, C13.P$1, C14.P$1, C15.P$1, J1.6, JP4.1, R13.P$2, R4.P$2, U1.FB, U2.VCC, U4.D2/, U4.SLEW
Other:
- note added: "aeg_driver (c) 2020 jjp@pobox.com Licensed under the Apache 2.0 License"
- moved on the sheet: C10, C11, C12, C13, C14, C15, C2, C3, C4, C5, C6, C7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

Commit message: aeg_driver: Curate BOM
Parts:
- C10, C4: value 10uF 35V -> 10uF 50V; MPN CGA5L1X7R1V106K160AC -> C3216X7R1H106K160AE
- C11, C5, C6, C7, C8, C9: HOUSEPART 1 -> YES
- J1, J2, J3, J4: POPULATE (none) -> 0
- J5: MPN (none) -> XT30PW-M; POPULATE 0 -> 1
Changed lines of the file:
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@@
 </part>
 <part name="J5" library="controller" deviceset="XT30" device="XT30PW_MALE">
-<attribute name="POPULATE" value="0"/>
+<attribute name="MPN" value="XT30PW-M"/>
+<attribute name="POPULATE" value="1"/>
 </part>
 <part name="P+5" library="supply1" deviceset="V+" device=""/>
@@
 </part>
 <part name="C5" library="mfpassives" deviceset="CAPACITOR_NP" device="_0402" value="0.1uF">
-<attribute name="HOUSEPART" value="1"/>
+<attribute name="HOUSEPART" value="YES"/>
 <attribute name="MPN" value="MF-CAP-0402-0.1uF"/>
 </part>
 <part name="C6" library="mfpassives" deviceset="CAPACITOR_NP" device="_0402" value="0.1uF">
-<attribute name="HOUSEPART" value="1"/>
+<attribute name="HOUSEPART" value="YES"/>
 <attribute name="MPN" value="MF-CAP-0402-0.1uF"/>
 </part>
 <part name="C11" library="mfpassives" deviceset="CAPACITOR_NP" device="_0402" value="0.1uF">
-<attribute name="HOUSEPART" value="1"/>
+<attribute name="HOUSEPART" value="YES"/>
 <attribute name="MPN" value="MF-CAP-0402-0.1uF"/>
 </part>
 <part name="C9" library="mfpassives" deviceset="CAPACITOR_NP" device="_0402" value="0.1uF">
-<attribute name="HOUSEPART" value="1"/>
+<attribute name="HOUSEPART" value="YES"/>
 <attribute name="MPN" value="MF-CAP-0402-0.1uF"/>
 </part>
 <part name="C8" library="mfpassives" deviceset="CAPACITOR_NP" device="_0402" value="0.1uF">
-<attribute name="HOUSEPART" value="1"/>
+<attribute name="HOUSEPART" value="YES"/>
 <attribute name="MPN" value="MF-CAP-0402-0.1uF"/>
 </part>
 <part name="C7" library="mfpassives" deviceset="CAPACITOR_NP" device="_0402" value="1uF">
-<attribute name="HOUSEPART" value="1"/>
+<attribute name="HOUSEPART" value="YES"/>
 <attribute name="MPN" value="MF-CAP-0402-1uF"/>
 </part>
-<part name="C10" library="mfpassives" deviceset="CAPACITOR_NP" device="_1206" value="10uF 35V">
-<attribute name="MF" value="TDK"/>
-<attribute name="MPN" value="CGA5L1X7R1V106K160AC"/>
+<part name="C10" library="mfpassives" deviceset="CAPACITOR_NP" device="_1206" value="10uF 50V">
+<attribute name="MF" value="TDK"/>
+<attribute name="MPN" value="C3216X7R1H106K160AE"/>
 </part>
 <part name="J6" library="precharge" deviceset="JST-ZH6" device="SMT_VERT">
@@
 <attribute name="POPULATE" value="1"/>
 </part>
-<part name="C4" library="mfpassives" deviceset="CAPACITOR_NP" device="_1206" value="10uF 35V">
-<attribute name="MF" value="TDK"/>
-<attribute name="MPN" value="CGA5L1X7R1V106K160AC"/>
+<part name="C4" library="mfpassives" deviceset="CAPACITOR_NP" device="_1206" value="10uF 50V">
+<attribute name="MF" value="TDK"/>
+<attribute name="MPN" value="C3216X7R1H106K160AE"/>
 </part>
 <part name="C2" library="mfpassives" deviceset="CAPACITOR_NP" device="_0603" value="1uF 50V">
@@
 </part>
 <part name="P+4" library="supply1" deviceset="V+" device=""/>
-<part name="J2" library="pinhead" library_urn="urn:adsk.eagle:library:325" deviceset="PINHD-1X2" device="" package3d_urn="urn:adsk.eagle:package:22435/2"/>
-<part name="J4" library="pinhead" library_urn="urn:adsk.eagle:library:325" deviceset="PINHD-1X2" device="" package3d_urn="urn:adsk.eagle:package:22435/2"/>
-<part name="J3" library="pinhead" library_urn="urn:adsk.eagle:library:325" deviceset="PINHD-1X2" device="" package3d_urn="urn:adsk.eagle:package:22435/2"/>
+<part name="J2" library="pinhead" library_urn="urn:adsk.eagle:library:325" deviceset="PINHD-1X2" device="" package3d_urn="urn:adsk.eagle:package:22435/2">
+<attribute name="POPULATE" value="0"/>
+</part>
+<part name="J4" library="pinhead" library_urn="urn:adsk.eagle:library:325" deviceset="PINHD-1X2" device="" package3d_urn="urn:adsk.eagle:package:22435/2">
+<attribute name="POPULATE" value="0"/>
+</part>
+<part name="J3" library="pinhead" library_urn="urn:adsk.eagle:library:325" deviceset="PINHD-1X2" device="" package3d_urn="urn:adsk.eagle:package:22435/2">
+<attribute name="POPULATE" value="0"/>
+</part>
 <part name="GND7" library="supply1" deviceset="GND" device=""/>
 <part name="U1" library="mfdiscrete" deviceset="N-CHANNEL_FET" device="_SOT-23-3">
@@
 <attribute name="POPULATE" value="1"/>
 </part>
-<part name="J1" library="pinhead" library_urn="urn:adsk.eagle:library:325" deviceset="PINHD-1X2" device="" package3d_urn="urn:adsk.eagle:package:22435/2"/>
+<part name="J1" library="pinhead" library_urn="urn:adsk.eagle:library:325" deviceset="PINHD-1X2" device="" package3d_urn="urn:adsk.eagle:package:22435/2">
+<attribute name="POPULATE" value="0"/>
+</part>
 <part name="GND8" library="supply1" deviceset="GND" device=""/>
 <part name="GND9" library="supply1" deviceset="GND" device=""/>
@@
 <attribute name="NAME" x="121.92" y="-42.418" size="1.778" layer="95"/>
 <attribute name="VALUE" x="121.92" y="-55.626" size="1.778" layer="96"/>
+<attribute name="MPN" x="127" y="-48.26" size="1.778" layer="96" font="vector" display="off"/>
 </instance>
 <instance part="P+5" gate="1" x="152.4" y="-38.1" smashed="yes">
@@
 <attribute name="NAME" x="359.41" y="-212.725" size="1.778" layer="95"/>
 <attribute name="VALUE" x="359.41" y="-223.52" size="1.778" layer="96"/>
+<attribute name="POPULATE" x="365.76" y="-218.44" size="1.778" layer="96" font="vector" display="off"/>
 </instance>
 <instance part="J4" gate="G$1" x="558.8" y="-203.2" smashed="yes">
 <attribute name="NAME" x="552.45" y="-197.485" size="1.778" layer="95"/>
 <attribute name="VALUE" x="552.45" y="-208.28" size="1.778" layer="96"/>
+<attribute name="POPULATE" x="558.8" y="-203.2" size="1.778" layer="96" font="vector" display="off"/>
 </instance>
 <instance part="J3" gate="G$1" x="558.8" y="-228.6" smashed="yes">
 <attribute name="NAME" x="552.45" y="-222.885" size="1.778" layer="95"/>
 <attribute name="VALUE" x="552.45" y="-233.68" size="1.778" layer="96"/>
+<attribute name="POPULATE" x="558.8" y="-228.6" size="1.778" layer="96" font="vector" display="off"/>
 </instance>
 <instance part="GND7" gate="1" x="68.58" y="-121.92" smashed="yes">
@@
 <attribute name="NAME" x="69.85" y="-85.725" size="1.778" layer="95"/>
 <attribute name="VALUE" x="69.85" y="-96.52" size="1.778" layer="96"/>
+<attribute name="POPULATE" x="76.2" y="-91.44" size="1.778" layer="96" font="vector" display="off"/>
 </instance>
 <instance part="GND8" gate="1" x="548.64" y="-233.68" smashed="yes">
